Commit message: Configured urdf files to work in ros2 with controller manager edited sim launch for testing wheel urdfs created rsp.wheel.py launch file for wheels for testing

File: src/icarus_pi/Mesh/Mecanum-Right/urdf/Mecanum-Right.urdf.xacro (robot description, xacro)
@@ -27,19 +27,19 @@
       <geometry>
         <mesh
-          filename="package://Mecanum-Right/meshes/Right_Base_Link.STL" />
-      </geometry>
-      <material
-        name="">
-        <color
-          rgba="0.792156862745098 0.819607843137255 0.933333333333333 1" />
-      </material>
-    </visual>
-    <collision>
-      <origin
-        xyz="0 0 0"
-        rpy="0 0 0" />
-      <geometry>
-        <mesh
-          filename="package://Mecanum-Right/meshes/Right_Base_Link.STL" />
+          filename="file://$(find icarus_pi)/Mesh/Mecanum-Right/meshes/Right_Base_Link.STL" />
+      </geometry>
+      <material
+        name="">
+        <color
+          rgba="0.792156862745098 0.819607843137255 0.933333333333333 1" />
+      </material>
+    </visual>
+    <collision>
+      <origin
+        xyz="0 0 0"
+        rpy="0 0 0" />
+      <geometry>
+        <mesh
+          filename="file://$(find icarus_pi)/Mesh/Mecanum-Right/meshes/Right_Base_Link.STL" />
       </geometry>
     </collision>
@@ -67,19 +67,19 @@
       <geometry>
         <mesh
-          filename="package://Mecanum-Right/meshes/Mecanum_Roller_Link1.STL" />
-      </geometry>
-      <material
-        name="">
-        <color
-          rgba="0.792156862745098 0.819607843137255 0.933333333333333 1" />
-      </material>
-    </visual>
-    <collision>
-      <origin
-        xyz="0 0 0"
-        rpy="0 0 0" />
-      <geometry>
-        <mesh
-          filename="package://Mecanum-Right/meshes/Mecanum_Roller_Link1.STL" />
+          filename="file://$(find icarus_pi)/Mesh/Mecanum-Right/meshes/Mecanum_Roller_Link1.STL" />
+      </geometry>
+      <material
+        name="">
+        <color
+          rgba="0.792156862745098 0.819607843137255 0.933333333333333 1" />
+      </material>
+    </visual>
+    <collision>
+      <origin
+        xyz="0 0 0"
+        rpy="0 0 0" />
+      <geometry>
+        <mesh
+          filename="file://$(find icarus_pi)/Mesh/Mecanum-Right/meshes/Mecanum_Roller_Link1.STL" />
       </geometry>
     </collision>
@@ -120,19 +120,19 @@
       <geometry>
         <mesh
-          filename="package://Mecanum-Right/meshes/Mecanum_Roller_Link2.STL" />
-      </geometry>
-      <material
-        name="">
-        <color
-          rgba="0.792156862745098 0.819607843137255 0.933333333333333 1" />
-      </material>
-    </visual>
-    <collision>
-      <origin
-        xyz="0 0 0"
-        rpy="0 0 0" />
-      <geometry>
-        <mesh
-          filename="package://Mecanum-Right/meshes/Mecanum_Roller_Link2.STL" />
+          filename="file://$(find icarus_pi)/Mesh/Mecanum-Right/meshes/Mecanum_Roller_Link2.STL" />
+      </geometry>
+      <material
+        name="">
+        <color
+          rgba="0.792156862745098 0.819607843137255 0.933333333333333 1" />
+      </material>
+    </visual>
+    <collision>
+      <origin
+        xyz="0 0 0"
+        rpy="0 0 0" />
+      <geometry>
+        <mesh
+          filename="file://$(find icarus_pi)/Mesh/Mecanum-Right/meshes/Mecanum_Roller_Link2.STL" />
       </geometry>
     </collision>
@@ -173,19 +173,19 @@
       <geometry>
         <mesh
-          filename="package://Mecanum-Right/meshes/Mecanum_Roller_Link3.STL" />
-      </geometry>
-      <material
-        name="">
-        <color
-          rgba="0.792156862745098 0.819607843137255 0.933333333333333 1" />
-      </material>
-    </visual>
-    <collision>
-      <origin
-        xyz="0 0 0"
-        rpy="0 0 0" />
-      <geometry>
-        <mesh
-          filename="package://Mecanum-Right/meshes/Mecanum_Roller_Link3.STL" />
+          filename="file://$(find icarus_pi)/Mesh/Mecanum-Right/meshes/Mecanum_Roller_Link3.STL" />
+      </geometry>
+      <material
+        name="">
+        <color
+          rgba="0.792156862745098 0.819607843137255 0.933333333333333 1" />
+      </material>
+    </visual>
+    <collision>
+      <origin
+        xyz="0 0 0"
+        rpy="0 0 0" />
+      <geometry>
+        <mesh
+          filename="file://$(find icarus_pi)/Mesh/Mecanum-Right/meshes/Mecanum_Roller_Link3.STL" />
       </geometry>
     </collision>
@@ -226,19 +226,19 @@
       <geometry>
         <mesh
-          filename="package://Mecanum-Right/meshes/Mecanum_Roller_Link4.STL" />
-      </geometry>
-      <material
-        name="">
-        <color
-          rgba="0.792156862745098 0.819607843137255 0.933333333333333 1" />
-      </material>
-    </visual>
-    <collision>
-      <origin
-        xyz="0 0 0"
-        rpy="0 0 0" />
-      <geometry>
-        <mesh
-          filename="package://Mecanum-Right/meshes/Mecanum_Roller_Link4.STL" />
+          filename="file://$(find icarus_pi)/Mesh/Mecanum-Right/meshes/Mecanum_Roller_Link4.STL" />
+      </geometry>
+      <material
+        name="">
+        <color
+          rgba="0.792156862745098 0.819607843137255 0.933333333333333 1" />
+      </material>
+    </visual>
+    <collision>
+      <origin
+        xyz="0 0 0"
+        rpy="0 0 0" />
+      <geometry>
+        <mesh
+          filename="file://$(find icarus_pi)/Mesh/Mecanum-Right/meshes/Mecanum_Roller_Link4.STL" />
       </geometry>
     </collision>
@@ -279,19 +279,19 @@
       <geometry>
         <mesh
-          filename="package://Mecanum-Right/meshes/Mecanum_Roller_Link5.STL" />
-      </geometry>
-      <material
-        name="">
-        <color
-          rgba="0.792156862745098 0.819607843137255 0.933333333333333 1" />
-      </material>
-    </visual>
-    <collision>
-      <origin
-        xyz="0 0 0"
-        rpy="0 0 0" />
-      <geometry>
-        <mesh
-          filename="package://Mecanum-Right/meshes/Mecanum_Roller_Link5.STL" />
+          filename="file://$(find icarus_pi)/Mesh/Mecanum-Right/meshes/Mecanum_Roller_Link5.STL" />
+      </geometry>
+      <material
+        name="">
+        <color
+          rgba="0.792156862745098 0.819607843137255 0.933333333333333 1" />
+      </material>
+    </visual>
+    <collision>
+      <origin
+        xyz="0 0 0"
+        rpy="0 0 0" />
+      <geometry>
+        <mesh
+          filename="file://$(find icarus_pi)/Mesh/Mecanum-Right/meshes/Mecanum_Roller_Link5.STL" />
       </geometry>
     </collision>
@@ -332,19 +332,19 @@
       <geometry>
         <mesh
-          filename="package://Mecanum-Right/meshes/Mecanum_Roller_Link6.STL" />
-      </geometry>
-      <material
-        name="">
-        <color
-          rgba="0.792156862745098 0.819607843137255 0.933333333333333 1" />
-      </material>
-    </visual>
-    <collision>
-      <origin
-        xyz="0 0 0"
-        rpy="0 0 0" />
-      <geometry>
-        <mesh
-          filename="package://Mecanum-Right/meshes/Mecanum_Roller_Link6.STL" />
+          filename="file://$(find icarus_pi)/Mesh/Mecanum-Right/meshes/Mecanum_Roller_Link6.STL" />
+      </geometry>
+      <material
+        name="">
+        <color
+          rgba="0.792156862745098 0.819607843137255 0.933333333333333 1" />
+      </material>
+    </visual>
+    <collision>
+      <origin
+        xyz="0 0 0"
+        rpy="0 0 0" />
+      <geometry>
+        <mesh
+          filename="file://$(find icarus_pi)/Mesh/Mecanum-Right/meshes/Mecanum_Roller_Link6.STL" />
       </geometry>
     </collision>
@@ -385,19 +385,19 @@
       <geometry>
         <mesh
-          filename="package://Mecanum-Right/meshes/Mecanum_Roller_Link7.STL" />
-      </geometry>
-      <material
-        name="">
-        <color
-          rgba="0.792156862745098 0.819607843137255 0.933333333333333 1" />
-      </material>
-    </visual>
-    <collision>
-      <origin
-        xyz="0 0 0"
-        rpy="0 0 0" />
-      <geometry>
-        <mesh
-          filename="package://Mecanum-Right/meshes/Mecanum_Roller_Link7.STL" />
+          filename="file://$(find icarus_pi)/Mesh/Mecanum-Right/meshes/Mecanum_Roller_Link7.STL" />
+      </geometry>
+      <material
+        name="">
+        <color
+          rgba="0.792156862745098 0.819607843137255 0.933333333333333 1" />
+      </material>
+    </visual>
+    <collision>
+      <origin
+        xyz="0 0 0"
+        rpy="0 0 0" />
+      <geometry>
+        <mesh
+          filename="file://$(find icarus_pi)/Mesh/Mecanum-Right/meshes/Mecanum_Roller_Link7.STL" />
       </geometry>
     </collision>
@@ -438,19 +438,19 @@
       <geometry>
         <mesh
-          filename="package://Mecanum-Right/meshes/Mecanum_Roller_Link8.STL" />
-      </geometry>
-      <material
-        name="">
-        <color
-          rgba="0.792156862745098 0.819607843137255 0.933333333333333 1" />
-      </material>
-    </visual>
-    <collision>
-      <origin
-        xyz="0 0 0"
-        rpy="0 0 0" />
-      <geometry>
-        <mesh
-          filename="package://Mecanum-Right/meshes/Mecanum_Roller_Link8.STL" />
+          filename="file://$(find icarus_pi)/Mesh/Mecanum-Right/meshes/Mecanum_Roller_Link8.STL" />
+      </geometry>
+      <material
+        name="">
+        <color
+          rgba="0.792156862745098 0.819607843137255 0.933333333333333 1" />
+      </material>
+    </visual>
+    <collision>
+      <origin
+        xyz="0 0 0"
+        rpy="0 0 0" />
+      <geometry>
+        <mesh
+          filename="file://$(find icarus_pi)/Mesh/Mecanum-Right/meshes/Mecanum_Roller_Link8.STL" />
       </geometry>
     </collision>
@@ -491,19 +491,19 @@
       <geometry>
         <mesh
-          filename="package://Mecanum-Right/meshes/Mecanum_Roller_Link9.STL" />
-      </geometry>
-      <material
-        name="">
-        <color
-          rgba="0.792156862745098 0.819607843137255 0.933333333333333 1" />
-      </material>
-    </visual>
-    <collision>
-      <origin
-        xyz="0 0 0"
-        rpy="0 0 0" />
-      <geometry>
-        <mesh
-          filename="package://Mecanum-Right/meshes/Mecanum_Roller_Link9.STL" />
+          filename="file://$(find icarus_pi)/Mesh/Mecanum-Right/meshes/Mecanum_Roller_Link9.STL" />
+      </geometry>
+      <material
+        name="">
+        <color
+          rgba="0.792156862745098 0.819607843137255 0.933333333333333 1" />
+      </material>
+    </visual>
+    <collision>
+      <origin
+        xyz="0 0 0"
+        rpy="0 0 0" />
+      <geometry>
+        <mesh
+          filename="file://$(find icarus_pi)/Mesh/Mecanum-Right/meshes/Mecanum_Roller_Link9.STL" />
       </geometry>
     </collision>
@@ -522,3 +522,88 @@
       xyz="1 0 0" />
   </joint>
+    <ros2_control name="gazeboSimSystem" type="system">
+		<hardware>
+			<plugin>gazebo_ros2_control/GazeboSystem</plugin>
+		</hardware>
+		<joint name="Mecanum_roller_joint_1">
+			<command_interface name="velocity">
+				<param name="min">-100</param>
+				<param name="max">100</param>
+			</command_interface>
+			<state_interface name="position"/>
+			<state_interface name="velocity"/>
+		</joint>
+		<joint name="Mecanum_roller_joint_2">
+			<command_interface name="velocity">
+				<param name="min">-100</param>
+				<param name="max">100</param>
+			</command_interface>
+			<state_interface name="position"/>
+			<state_interface name="velocity"/>
+		</joint>
+    		<joint name="Mecanum_roller_joint_3">
+			<command_interface name="velocity">
+				<param name="min">-100</param>
+				<param name="max">100</param>
+			</command_interface>
+			<state_interface name="position"/>
+			<state_interface name="velocity"/>
+		</joint>
+    		<joint name="Mecanum_roller_joint_4">
+			<command_interface name="velocity">
+				<param name="min">-100</param>
+				<param name="max">100</param>
+			</command_interface>
+			<state_interface name="position"/>
+			<state_interface name="velocity"/>
+		</joint>
+    		<joint name="Mecanum_roller_joint_5">
+			<command_interface name="velocity">
+				<param name="min">-100</param>
+				<param name="max">100</param>
+			</command_interface>
+			<state_interface name="position"/>
+			<state_interface name="velocity"/>
+		</joint>
+    		<joint name="Mecanum_roller_joint_6">
+			<command_interface name="velocity">
+				<param name="min">-100</param>
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