Commit message: Wheel orientation corrected

File: src/icarus_pi/description/Mecanum.urdf.xacro (robot description, xacro)
@@ -1,42 +1,42 @@
-<?xml version="1.0" encoding="utf-8"?>
+<?xml version="1.0"?>
 <robot xmlns:xacro="http://www.ros.org/wiki/xacro" >
-  <xacro:macro name="MecanumR" params="prefix x_reflect y_reflect">
+  <xacro:macro name="Mecanum" params="prefix x_reflect y_reflect r_reflect">
   <link
     name="${prefix}_link">
     <inertial>
       <origin
-        xyz="-4.7771233839358E-07 2.34552518933002E-07 -2.07119508697187E-07"
-        rpy="0 0 0" />
-      <mass
-        value="0.0110925597603562" />
-      <inertia
-        ixx="1.26410691718137E-06"
-        ixy="-1.5460162528858E-07"
-        ixz="1.36519585539842E-07"
-        iyy="1.02513832514045E-06"
-        iyz="-6.70299050271453E-08"
-        izz="1.00842045851304E-06" />
-    </inertial>
-    <visual>
-      <origin
-        xyz="0 0 0"
-        rpy="0 0 0" />
-      <geometry>
-        <mesh
-          filename="file://$(find icarus_pi)/Mesh/Mecanum-Right/meshes/Right_Base_Link.STL" />
-      </geometry>
-      <material
-        name="">
-        <color
-          rgba="0.792156862745098 0.819607843137255 0.933333333333333 1" />
-      </material>
-    </visual>
-    <collision>
-      <origin
-        xyz="0 0 0"
-        rpy="0 0 0" />
-      <geometry>
-        <mesh
-          filename="file://$(find icarus_pi)/Mesh/Mecanum-Right/meshes/Right_Base_Link.STL" />
+        xyz="-5.71071320654166E-07 1.24074703998625E-17 -8.40087960733809E-19"
+        rpy="0 0 0" />
+      <mass
+        value="0.0110925597603563" />
+      <inertia
+        ixx="1.39920510272198E-06"
+        ixy="6.03598608368132E-22"
+        ixz="2.70201401925188E-21"
+        iyy="9.49230299056441E-07"
+        iyz="-8.48228743085689E-23"
+        izz="9.49230299056441E-07" />
+    </inertial>
+    <visual>
+      <origin
+        xyz="0 0 0"
+        rpy="0 0 0" />
+      <geometry>
+        <mesh
+          filename="file://$(find icarus_pi)/Mesh/Mecanum-Left/meshes/base_link.STL" />
+      </geometry>
+      <material
+        name="">
+        <color
+          rgba="0.792156862745098 0.819607843137255 0.933333333333333 1" />
+      </material>
+    </visual>
+    <collision>
+      <origin
+        xyz="0 0 0"
+        rpy="0 0 0" />
+      <geometry>
+        <mesh
+          filename="file://$(find icarus_pi)/Mesh/Mecanum-Left/meshes/base_link.STL" />
       </geometry>
     </collision>
@@ -45,12 +45,329 @@
 		<parent link="base_link"/>
 		<child link="${prefix}_link"/>
-		<origin xyz="${x_reflect*wheel_xoff} ${y_reflect*(chassis_width/2 + wheel_ygap)} ${-wheel_zoff}" rpy="0 0 0"/>
-    <axis xyz="0 0 1"/>
+		<origin xyz="${x_reflect*wheel_xoff} ${y_reflect*(chassis_width/2 + wheel_ygap)} ${-wheel_zoff}" rpy="0 0 ${r_reflect}"/>
+    <axis xyz="1 0 0"/>
 	</joint>
   <link
-    name="${prefix}_Mecanum_Roller_Link1">
-    <inertial>
-      <origin
-        xyz="-4.16595979552251E-05 0 1.56125112837913E-17"
+    name="${prefix}_Mecanum_roller_link_1">
+    <inertial>
+      <origin
+        xyz="4.19537259525784E-05 -9.19403442267708E-17 -4.5102810375397E-17"
+        rpy="0 0 0" />
+      <mass
+        value="0.00104310145784987" />
+      <inertia
+        ixx="9.96758957260103E-09"
+        ixy="8.47860127866853E-24"
+        ixz="-4.54949336904165E-24"
+        iyy="3.79225492604175E-08"
+        iyz="3.30872245021211E-24"
+        izz="3.79225492604176E-08" />
+    </inertial>
+    <visual>
+      <origin
+        xyz="0 0 0"
+        rpy="0 0 0" />
+      <geometry>
+        <mesh
+          filename="file://$(find icarus_pi)/Mesh/Mecanum-Left/meshes/Mecanum_roller_link_1.STL" />
+      </geometry>
+      <material
+        name="">
+        <color
+          rgba="0.792156862745098 0.819607843137255 0.933333333333333 1" />
+      </material>
+    </visual>
+    <collision>
+      <origin
+        xyz="0 0 0"
+        rpy="0 0 0" />
+      <geometry>
+        <mesh
+          filename="file://$(find icarus_pi)/Mesh/Mecanum-Left/meshes/Mecanum_roller_link_1.STL" />
+      </geometry>
+    </collision>
+  </link>
+  <joint
+    name="${prefix}_Mecanum_roller_joint_1" type="continuous">
+    <origin
+      xyz="0.00012912 0.014344 0.0095825"
+      rpy="-2.7656 0.6249 2.6298" />
+    <parent
+      link="${prefix}_link" />
+    <child
+      link="${prefix}_Mecanum_roller_link_1" />
+    <axis
+      xyz="1 0 0" />
+  </joint>
+  <link
+    name="${prefix}_Mecanum_roller_link_2">
+    <inertial>
+      <origin
+        xyz="-4.19537259514885E-05 -2.77555756156289E-17 -9.71445146547012E-17"
+        rpy="0 0 0" />
+      <mass
+        value="0.00104310145784987" />
+      <inertia
+        ixx="9.96758957260103E-09"
+        ixy="1.68021061924834E-24"
+        ixz="-5.37667398159468E-24"
+        iyy="3.79225492604175E-08"
+        iyz="-1.03397576569128E-25"
+        izz="3.79225492604175E-08" />
+    </inertial>
+    <visual>
+      <origin
+        xyz="0 0 0"
+        rpy="0 0 0" />
+      <geometry>
+        <mesh
+          filename="file://$(find icarus_pi)/Mesh/Mecanum-Left/meshes/Mecanum_roller_link_2.STL" />
+      </geometry>
+      <material
+        name="">
+        <color
+          rgba="0.792156862745098 0.819607843137255 0.933333333333333 1" />
+      </material>
+    </visual>
+    <collision>
+      <origin
+        xyz="0 0 0"
+        rpy="0 0 0" />
+      <geometry>
+        <mesh
+          filename="file://$(find icarus_pi)/Mesh/Mecanum-Left/meshes/Mecanum_roller_link_2.STL" />
+      </geometry>
+    </collision>
+  </link>
+  <joint
+    name="${prefix}_Mecanum_roller_joint_2"
+    type="continuous">
+    <origin
+      xyz="-0.00012933 0.0045802 0.016631"
+      rpy="1.6775 -0.19406 -0.76608" />
+    <parent
+      link="${prefix}_link" />
+    <child
+      link="${prefix}_Mecanum_roller_link_2" />
+    <axis
+      xyz="1 0 0" />
+  </joint>
+  <link
+    name="${prefix}_Mecanum_roller_link_3">
+    <inertial>
+      <origin
+        xyz="-4.19537259517232E-05 6.24500451351651E-17 -1.45716771982052E-16"
+        rpy="0 0 0" />
+      <mass
+        value="0.00104310145784987" />
+      <inertia
+        ixx="9.96758957260103E-09"
+        ixy="4.39439700418796E-24"
+        ixz="-8.27180612553028E-25"
+        iyy="3.79225492604175E-08"
+        iyz="-1.65436122510606E-24"
+        izz="3.79225492604175E-08" />
+    </inertial>
+    <visual>
+      <origin
+        xyz="0 0 0"
+        rpy="0 0 0" />
+      <geometry>
+        <mesh
+          filename="file://$(find icarus_pi)/Mesh/Mecanum-Left/meshes/Mecanum_roller_link_3.STL" />
+      </geometry>
+      <material
+        name="">
+        <color
+          rgba="0.792156862745098 0.819607843137255 0.933333333333333 1" />
+      </material>
+    </visual>
+    <collision>
+      <origin
+        xyz="0 0 0"
+        rpy="0 0 0" />
+      <geometry>
+        <mesh
+          filename="file://$(find icarus_pi)/Mesh/Mecanum-Left/meshes/Mecanum_roller_link_3.STL" />
+      </geometry>
+    </collision>
+  </link>
+  <joint
+    name="${prefix}_Mecanum_roller_joint_3"
+    type="continuous">
+    <origin
+      xyz="0.00012912 -0.006946 0.01579"
+      rpy="1.4846 0.29377 -0.73958" />
+    <parent
+      link="${prefix}_link" />
+    <child
+      link="${prefix}_Mecanum_roller_link_3" />
+    <axis
+      xyz="1 0 0" />
+  </joint>
+  <link
+    name="${prefix}_Mecanum_roller_link_4">
+    <inertial>
+      <origin
+        xyz="-4.19537259518845E-05 9.54097911787244E-17 -5.03069808033274E-17"
+        rpy="0 0 0" />
+      <mass
+        value="0.00104310145784987" />
+      <inertia
+        ixx="9.9675895729459E-09"
+        ixy="-5.11818004017186E-24"
+        ixz="2.68833699079734E-24"
+        iyy="3.79225492606102E-08"
+        iyz="-8.27180612553028E-25"
+        izz="3.79225492606102E-08" />
+    </inertial>
+    <visual>
+      <origin
+        xyz="0 0 0"
+        rpy="0 0 0" />
+      <geometry>
+        <mesh
+          filename="file://$(find icarus_pi)/Mesh/Mecanum-Left/meshes/Mecanum_roller_link_4.STL" />
+      </geometry>
+      <material
+        name="">
+        <color
+          rgba="0.792156862745098 0.819607843137255 0.933333333333333 1" />
+      </material>
+    </visual>
+    <collision>
+      <origin
+        xyz="0 0 0"
+        rpy="0 0 0" />
+      <geometry>
+        <mesh
+          filename="file://$(find icarus_pi)/Mesh/Mecanum-Left/meshes/Mecanum_roller_link_4.STL" />
+      </geometry>
+    </collision>
+  </link>
+  <joint
+    name="${prefix}_Mecanum_roller_joint_4"
+    type="continuous">
+    <origin
+      xyz="0.00012912 -0.015471 0.0076312"
+      rpy="1.4497 0.68992 -0.41086" />
+    <parent
+      link="${prefix}_link" />
+    <child
+      link="${prefix}_Mecanum_roller_link_4" />
+    <axis
+      xyz="1 0 0" />
+  </joint>
+  <link
+    name="${prefix}_Mecanum_roller_link_5">
+    <inertial>
+      <origin
+        xyz="4.1659597956364E-05 1.04950770296597E-16 1.38777878078145E-17"
+        rpy="0 0 0" />
+      <mass
+        value="0.00104310145784987" />
+      <inertia
+        ixx="9.96758957260103E-09"
+        ixy="3.87740912134232E-25"
+        ixz="-2.1713491079517E-24"
+        iyy="3.79225492604175E-08"
+        iyz="2.06795153138257E-25"
+        izz="3.79225492604175E-08" />
+    </inertial>
+    <visual>
+      <origin
+        xyz="0 0 0"
+        rpy="0 0 0" />
+      <geometry>
+        <mesh
+          filename="file://$(find icarus_pi)/Mesh/Mecanum-Left/meshes/Mecanum_roller_link_5.STL" />
+      </geometry>
+      <material
+        name="">
+        <color
+          rgba="0.792156862745098 0.819607843137255 0.933333333333333 1" />
+      </material>
+    </visual>
+    <collision>
+      <origin
+        xyz="0 0 0"
+        rpy="0 0 0" />
+      <geometry>
+        <mesh
+          filename="file://$(find icarus_pi)/Mesh/Mecanum-Left/meshes/Mecanum_roller_link_5.STL" />
+      </geometry>
+    </collision>
+  </link>
+  <joint
+    name="${prefix}_Mecanum_roller_joint_5"
+    type="continuous">
+    <origin
+      xyz="0.00012912 -0.016757 -0.0040986"
+      rpy="1.6948 0.7554 0.24013" />
+    <parent
+      link="${prefix}_link" />
+    <child
+      link="${prefix}_Mecanum_roller_link_5" />
+    <axis
+      xyz="1 0 0" />
+  </joint>
+  <link
+    name="${prefix}_Mecanum_roller_link_6">
+    <inertial>
+      <origin
+        xyz="-4.19537259515289E-05 6.93889390390723E-18 1.73472347597681E-18"
+        rpy="0 0 0" />
+      <mass
+        value="0.00104310145784984" />
+      <inertia
+        ixx="9.96758957158561E-09"
+        ixy="-6.04875822929401E-24"
+        ixz="-1.15805285757424E-23"
+        iyy="3.79225492599098E-08"
+        iyz="8.27180612553028E-25"
+        izz="3.79225492599098E-08" />
+    </inertial>
+    <visual>
+      <origin
+        xyz="0 0 0"
+        rpy="0 0 0" />
+      <geometry>
+        <mesh
+          filename="file://$(find icarus_pi)/Mesh/Mecanum-Left/meshes/Mecanum_roller_link_6.STL" />
+      </geometry>
+      <material
+        name="">
+        <color
+          rgba="0.792156862745098 0.819607843137255 0.933333333333333 1" />
+      </material>
+    </visual>
+    <collision>
+      <origin
+        xyz="0 0 0"
+        rpy="0 0 0" />
+      <geometry>
+        <mesh
+          filename="file://$(find icarus_pi)/Mesh/Mecanum-Left/meshes/Mecanum_roller_link_6.STL" />
+      </geometry>
+    </collision>
+  </link>
+  <joint
+    name="${prefix}_Mecanum_roller_joint_6"
+    type="continuous">
+    <origin
+      xyz="0.00012912 -0.010202 -0.013911"
+      rpy="1.7524 0.42673 0.68129" />
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
File: src/icarus_pi/description/lidar.xacro (robot description, xacro)
@@ -15,5 +15,5 @@
 		</collision>
 		<visual>
-			<origin xyz = "${-chassis_length/2 + 2*lidar_radius} 0 ${chassis_height/4}" rpy="0 0 0"/>
+			<origin xyz = "${-chassis_length/2 + 2*lidar_radius} 0 ${chassis_height/16}" rpy="0 0 0"/>
 			<geometry>
 				<cylinder radius="${lidar_radius}" length=".06"/>
@@ -29,5 +29,5 @@
 		<parent link="base_link"/>
 		<child link="lidar_link"/>
-		<origin xyz="${-chassis_length/2 + lidar_radius} 0 ${chassis_height/2+.02}" rpy="0 0 0"/>
+		<origin xyz="${-chassis_length/2 + lidar_radius} 0 ${chassis_height/2+.03}" rpy="0 0 0"/>
 	</joint>
     <!--adding gazebo plugins to the sim-->

File: src/icarus_pi/description/robot_core.xacro (robot description, xacro)
@@ -42,9 +42,8 @@
     </gazebo>
      <!-- CHASSIS LINK -->
-    <xacro:include filename="Mecanum-Left.urdf.xacro"/>
-    <xacro:MecanumL prefix="frontRight" x_reflect="-1" y_reflect="1"/>
-    <xacro:MecanumL prefix="backLeft" x_reflect="1" y_reflect="-1"/>
-    <xacro:include filename="Mecanum-Right.urdf.xacro"/>
-    <xacro:MecanumR prefix="frontLeft" x_reflect="-1" y_reflect="-1"/>
-    <xacro:MecanumR prefix="backRight" x_reflect="1" y_reflect="1"/>
+    <xacro:include filename="Mecanum.urdf.xacro"/>
+    <xacro:Mecanum prefix="frontRight" x_reflect="-1" y_reflect="1" r_reflect="${pi/2}"/>
+    <xacro:Mecanum prefix="backLeft" x_reflect="1" y_reflect="-1" r_reflect="${pi/2}"/>
+    <xacro:Mecanum prefix="frontLeft" x_reflect="-1" y_reflect="-1" r_reflect="${pi/2}"/>
+    <xacro:Mecanum prefix="backRight" x_reflect="1" y_reflect="1" r_reflect="${pi/2}"/>
 </robot>

File: src/icarus_pi/description/robot_dimensions.xacro (robot description, xacro)
@@ -5,5 +5,5 @@
     <xacro:property name="chassis_width" value = ".203"/>
     <xacro:property name="chassis_height" value = ".16"/>
-    <xacro:property name="chassis_mass" value = "1"/>
+    <xacro:property name="chassis_mass" value = "10"/>
     <xacro:property name="wheel_radius" value = ".024"/>
     <xacro:property name="wheel_width" value = ".03"/>
