Commit message: reset head to early commit

File: src/icarus_pi/description/Mecanum.urdf.xacro (robot description, xacro)
@@ -6,15 +6,15 @@
     <inertial>
       <origin
-        xyz="-5.71071320654166E-07 1.24074703998625E-17 -8.40087960733809E-19"
-        rpy="0 0 0" />
-      <mass
-        value="0.0110925597603563" />
-      <inertia
-        ixx="1.39920510272198E-06"
-        ixy="6.03598608368132E-22"
-        ixz="2.70201401925188E-21"
-        iyy="9.49230299056441E-07"
-        iyz="-8.48228743085689E-23"
-        izz="9.49230299056441E-07" />
+        xyz="0.011813 0.0074643 0.015042"
+        rpy="0 0 0" />
+      <mass
+        value="0.010056" />
+      <inertia
+        ixx="1.2854E-06"
+        ixy="-1.0402E-23"
+        ixz="-1.8029E-21"
+        iyy="9.0867E-07"
+        iyz="-3.7562E-23"
+        izz="9.0867E-07" />
     </inertial>
     <visual>
@@ -29,5 +29,5 @@
         name="">
         <color
-          rgba="0.792156862745098 0.819607843137255 0.933333333333333 1" />
+          rgba="0.79216 0.81961 0.93333 1" />
       </material>
     </visual>
@@ -42,25 +42,25 @@
     </collision>
   </link>
-  <joint name="${prefix}_joint" type="continuous">
-		<parent link="base_link"/>
-		<child link="${prefix}_link"/>
-		<origin xyz="${x_reflect*wheel_xoff} ${y_reflect*(chassis_width/2 + wheel_ygap)} ${-wheel_zoff}" rpy="0 0 ${r_reflect}"/>
+    <joint name="${prefix}_joint" type="continuous">
+              <parent link="base_link"/>
+              <child link="${prefix}_link"/>
+              <origin xyz="${x_reflect*wheel_xoff} ${y_reflect*(chassis_width/2 + wheel_ygap)} ${-wheel_zoff}" rpy="0 0 ${r_reflect}"/>
     <axis xyz="1 0 0"/>
-	</joint>
-  <link
-    name="${prefix}_Mecanum_roller_link_1">
-    <inertial>
-      <origin
-        xyz="4.19537259525784E-05 -9.19403442267708E-17 -4.5102810375397E-17"
-        rpy="0 0 0" />
-      <mass
-        value="0.00104310145784987" />
-      <inertia
-        ixx="9.96758957260103E-09"
-        ixy="8.47860127866853E-24"
-        ixz="-4.54949336904165E-24"
-        iyy="3.79225492604175E-08"
-        iyz="3.30872245021211E-24"
-        izz="3.79225492604176E-08" />
+        </joint>
+  <link
+    name="Mecanum_roller_link_1">
+    <inertial>
+      <origin
+        xyz="0.012194 1.7694E-16 -2.3592E-16"
+        rpy="0 0 0" />
+      <mass
+        value="0.0010939" />
+      <inertia
+        ixx="1.1179E-08"
+        ixy="1.3442E-24"
+        ixz="4.1359E-25"
+        iyy="3.946E-08"
+        iyz="-2.068E-24"
+        izz="3.946E-08" />
     </inertial>
     <visual>
@@ -75,5 +75,5 @@
         name="">
         <color
-          rgba="0.792156862745098 0.819607843137255 0.933333333333333 1" />
+          rgba="0.79216 0.81961 0.93333 1" />
       </material>
     </visual>
@@ -91,6 +91,6 @@
     name="${prefix}_Mecanum_roller_joint_1" type="continuous">
     <origin
-      xyz="0.00012912 0.014344 0.0095825"
-      rpy="-2.7656 0.6249 2.6298" />
+      xyz="0.0032354879777911 -0.0211628583855368 0.0257385293646238"
+      rpy="1.40087787206783 0.523598775598295 -0.615479708670392" />
     <parent
       link="${prefix}_link" />
@@ -104,15 +104,15 @@
     <inertial>
       <origin
-        xyz="-4.19537259514885E-05 -2.77555756156289E-17 -9.71445146547012E-17"
-        rpy="0 0 0" />
-      <mass
-        value="0.00104310145784987" />
-      <inertia
-        ixx="9.96758957260103E-09"
-        ixy="1.68021061924834E-24"
-        ixz="-5.37667398159468E-24"
-        iyy="3.79225492604175E-08"
-        iyz="-1.03397576569128E-25"
-        izz="3.79225492604175E-08" />
+        xyz="0.0029529 -4.3368E-18 1.0408E-17"
+        rpy="0 0 0" />
+      <mass
+        value="0.0010939" />
+      <inertia
+        ixx="1.1179E-08"
+        ixy="-3.6706E-24"
+        ixz="-3.3087E-24"
+        iyy="3.946E-08"
+        iyz="0"
+        izz="3.946E-08" />
     </inertial>
     <visual>
@@ -127,5 +127,5 @@
         name="">
         <color
-          rgba="0.792156862745098 0.819607843137255 0.933333333333333 1" />
+          rgba="0.79216 0.81961 0.93333 1" />
       </material>
     </visual>
@@ -144,6 +144,6 @@
     type="continuous">
     <origin
-      xyz="-0.00012933 0.0045802 0.016631"
-      rpy="1.6775 -0.19406 -0.76608" />
+      xyz="0.013855 -0.025783 -0.0061895"
+      rpy="1.3738 -0.5236 -2.5261" />
     <parent
       link="${prefix}_link" />
@@ -157,15 +157,15 @@
     <inertial>
       <origin
-        xyz="-4.19537259517232E-05 6.24500451351651E-17 -1.45716771982052E-16"
-        rpy="0 0 0" />
-      <mass
-        value="0.00104310145784987" />
-      <inertia
-        ixx="9.96758957260103E-09"
-        ixy="4.39439700418796E-24"
-        ixz="-8.27180612553028E-25"
-        iyy="3.79225492604175E-08"
-        iyz="-1.65436122510606E-24"
-        izz="3.79225492604175E-08" />
+        xyz="-0.0023361 1.3878E-17 6.9389E-18"
+        rpy="0 0 0" />
+      <mass
+        value="0.0010939" />
+      <inertia
+        ixx="1.1179E-08"
+        ixy="1.4362E-22"
+        ixz="-4.26E-23"
+        iyy="3.946E-08"
+        iyz="-4.1359E-24"
+        izz="3.946E-08" />
     </inertial>
     <visual>
@@ -180,5 +180,5 @@
         name="">
         <color
-          rgba="0.792156862745098 0.819607843137255 0.933333333333333 1" />
+          rgba="0.79216 0.81961 0.93333 1" />
       </material>
     </visual>
@@ -197,6 +197,6 @@
     type="continuous">
     <origin
-      xyz="0.00012912 -0.006946 0.01579"
-      rpy="1.4846 0.29377 -0.73958" />
+      xyz="0.0134188663284221 -0.0134188663284221 -0.00978574865900883"
+      rpy="1.84520374289531 0 0.78539816339745" />
     <parent
       link="${prefix}_link" />
@@ -210,15 +210,15 @@
     <inertial>
       <origin
-        xyz="-4.19537259518845E-05 9.54097911787244E-17 -5.03069808033274E-17"
-        rpy="0 0 0" />
-      <mass
-        value="0.00104310145784987" />
-      <inertia
-        ixx="9.9675895729459E-09"
-        ixy="-5.11818004017186E-24"
-        ixz="2.68833699079734E-24"
-        iyy="3.79225492606102E-08"
-        iyz="-8.27180612553028E-25"
-        izz="3.79225492606102E-08" />
+        xyz="0.0030222 0 2.0817E-17"
+        rpy="0 0 0" />
+      <mass
+        value="0.0010939" />
+      <inertia
+        ixx="1.1179E-08"
+        ixy="-3.2743E-23"
+        ixz="-1.4241E-22"
+        iyy="3.946E-08"
+        iyz="-8.2718E-25"
+        izz="3.946E-08" />
     </inertial>
     <visual>
@@ -233,5 +233,5 @@
         name="">
         <color
-          rgba="0.792156862745098 0.819607843137255 0.933333333333333 1" />
+          rgba="0.79216 0.81961 0.93333 1" />
       </material>
     </visual>
@@ -250,6 +250,6 @@
     type="continuous">
     <origin
-      xyz="0.00012912 -0.015471 0.0076312"
-      rpy="1.4497 0.68992 -0.41086" />
+      xyz="0.00963 -0.032292 0.00963"
+      rpy="1.7863 0.7854 0" />
     <parent
       link="${prefix}_link" />
@@ -263,15 +263,15 @@
     <inertial>
       <origin
-        xyz="4.1659597956364E-05 1.04950770296597E-16 1.38777878078145E-17"
-        rpy="0 0 0" />
-      <mass
-        value="0.00104310145784987" />
-      <inertia
-        ixx="9.96758957260103E-09"
-        ixy="3.87740912134232E-25"
-        ixz="-2.1713491079517E-24"
-        iyy="3.79225492604175E-08"
-        iyz="2.06795153138257E-25"
-        izz="3.79225492604175E-08" />
+        xyz="0.013578 2.8623E-17 -7.546E-17"
+        rpy="0 0 0" />
+      <mass
+        value="0.0010939" />
+      <inertia
+        ixx="1.1179E-08"
+        ixy="-3.4704E-23"
+        ixz="1.4829E-22"
+        iyy="3.946E-08"
+        iyz="-8.2718E-25"
+        izz="3.946E-08" />
     </inertial>
     <visual>
@@ -286,5 +286,5 @@
         name="">
         <color
-          rgba="0.792156862745098 0.819607843137255 0.933333333333333 1" />
+          rgba="0.79216 0.81961 0.93333 1" />
       </material>
     </visual>
@@ -303,10 +303,10 @@
     type="continuous">
     <origin
-      xyz="0.00012912 -0.016757 -0.0040986"
-      rpy="1.6948 0.7554 0.24013" />
-    <parent
-      link="${prefix}_link" />
-    <child
-      link="${prefix}_Mecanum_roller_link_5" />
+      xyz="0.0021658 0.002208 -0.0021658"
+      rpy="1.2964 -0.7854 0" />
+    <parent
+      link="${prefix}_link" />
+    <child
+      link="${prefix}_Mecanum_roller_joint_5" />
     <axis
       xyz="1 0 0" />
@@ -316,15 +316,15 @@
     <inertial>
       <origin
-        xyz="-4.19537259515289E-05 6.93889390390723E-18 1.73472347597681E-18"
-        rpy="0 0 0" />
-      <mass
-        value="0.00104310145784984" />
-      <inertia
-        ixx="9.96758957158561E-09"
-        ixy="-6.04875822929401E-24"
-        ixz="-1.15805285757424E-23"
-        iyy="3.79225492599098E-08"
-        iyz="8.27180612553028E-25"
-        izz="3.79225492599098E-08" />
+        xyz="0.0045113 1.2143E-17 1.7347E-18"
+        rpy="0 0 0" />
+      <mass
+        value="0.0010939" />
+      <inertia
+        ixx="1.1179E-08"
+        ixy="-3.8774E-24"
+        ixz="0"
+        iyy="3.946E-08"
+        iyz="-1.6544E-24"
+        izz="3.946E-08" />
     </inertial>
     <visual>
@@ -339,5 +339,5 @@
         name="">
         <color
-          rgba="0.792156862745098 0.819607843137255 0.933333333333333 1" />
+          rgba="0.79216 0.81961 0.93333 1" />
       </material>
     </visual>
@@ -356,6 +356,6 @@
     type="continuous">
     <origin
-      xyz="0.00012912 -0.010202 -0.013911"
-      rpy="1.7524 0.42673 0.68129" />
+      xyz="0.00857701202220883 -0.00512037328736673 -0.00700935343907806"
+      rpy="1.40087787206783 -0.523598775598296 0.615479708670392" />
     <parent
       link="${prefix}_link" />
@@ -369,15 +369,15 @@
     <inertial>
       <origin
-        xyz="-4.19537259513104E-05 6.24500451351651E-17 4.16333634234434E-17"
-        rpy="0 0 0" />
-      <mass
-        value="0.00104310145784987" />
-      <inertia
-        ixx="9.96758957260102E-09"
-        ixy="-3.30872245021211E-24"
-        ixz="-1.03397576569128E-24"
-        iyy="3.79225492604175E-08"
-        iyz="2.48154183765908E-24"
-        izz="3.79225492604175E-08" />
+        xyz="0.018106 -5.2042E-18 3.4694E-18"
+        rpy="0 0 0" />
+      <mass
+        value="0.0010939" />
+      <inertia
+        ixx="1.1179E-08"
+        ixy="3.6189E-24"
+        ixz="-4.1359E-25"
+        iyy="3.946E-08"
+        iyz="0"
+        izz="3.946E-08" />
     </inertial>
     <visual>
@@ -392,5 +392,5 @@
         name="">
         <color
-          rgba="0.792156862745098 0.819607843137255 0.933333333333333 1" />
+          rgba="0.79216 0.81961 0.93333 1" />
       </material>
     </visual>
@@ -409,6 +409,6 @@
     type="continuous">
     <origin
-      xyz="0.00012912 0.0011266 -0.017214"
-      rpy="2.5112 -0.051481 0.78407" />
+      xyz="-0.0010359 0.006229 0.010588"
+      rpy="1.5572 -0.5236 -0.61548" />
     <parent
       link="${prefix}_link" />
@@ -422,15 +422,15 @@
     <inertial>
       <origin
-        xyz="4.16595979570254E-05 -8.67361737988404E-18 -6.93889390390723E-18"
-        rpy="0 0 0" />
-      <mass
-        value="0.00104310145784987" />
-      <inertia
-        ixx="9.96758957226301E-09"
-        ixy="-4.23930063933427E-24"
-        ixz="-3.30872245021211E-24"
-        iyy="3.79225492602485E-08"
-        iyz="-4.13590306276514E-25"
-        izz="3.79225492602485E-08" />
+        xyz="0 0 0"
+        rpy="0 0 0" />
+      <mass
+        value="0.001" />
+      <inertia
+        ixx="0"
+        ixy="0"
+        ixz="0"
+        iyy="0"
+        iyz="0"
+        izz="0" />
     </inertial>
     <visual>
@@ -445,5 +445,5 @@
         name="">
         <color
-          rgba="0.792156862745098 0.819607843137255 0.933333333333333 1" />
+          rgba="1 1 1 1" />
       </material>
     </visual>
@@ -462,63 +462,10 @@
     type="continuous">
     <origin
-      xyz="-0.00012933 0.012113 -0.012282"
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