Commit message: Added Mecanum to Robot Core

File: src/icarus_pi/description/Mecanum-Left.urdf.xacro (robot description, xacro)
@@ -1,6 +1,7 @@
 <?xml version="1.0"?>
-<robot name="Mecanum-Left" xmlns:xacro="http://www.ros.org/wiki/xacro" >
-  <link
-    name="base_link">
+<robot xmlns:xacro="http://www.ros.org/wiki/xacro" >
+  <xacro:macro name="MecanumL" params="prefix x_reflect y_reflect">
+  <link
+    name="${prefix}_link">
     <inertial>
       <origin
@@ -41,6 +42,12 @@
     </collision>
   </link>
-  <link
-    name="Mecanum_roller_link_1">
+  <joint name="${prefix}_joint" type="continuous">
+		<parent link="base_link"/>
+		<child link="${prefix}_link"/>
+		<origin xyz="${x_reflect*wheel_xoff} ${y_reflect*(chassis_width/2 + wheel_ygap)} ${-wheel_zoff}" rpy="${pi/2} 0 0"/>
+    <axis xyz="0 0 1"/>
+	</joint>
+  <link
+    name="${prefix}_Mecanum_roller_link_1">
     <inertial>
       <origin
@@ -82,18 +89,17 @@
   </link>
   <joint
-    name="Mecanum_roller_joint_1"
-    type="continuous">
+    name="${prefix}_Mecanum_roller_joint_1" type="continuous">
     <origin
       xyz="0.00012912 0.014344 0.0095825"
       rpy="-2.7656 0.6249 2.6298" />
     <parent
-      link="base_link" />
-    <child
-      link="Mecanum_roller_link_1" />
-    <axis
-      xyz="1 0 0" />
-  </joint>
-  <link
-    name="Mecanum_roller_link_2">
+      link="${prefix}_link" />
+    <child
+      link="${prefix}_Mecanum_roller_link_1" />
+    <axis
+      xyz="1 0 0" />
+  </joint>
+  <link
+    name="${prefix}_Mecanum_roller_link_2">
     <inertial>
       <origin
@@ -135,5 +141,5 @@
   </link>
   <joint
-    name="Mecanum_roller_joint_2"
+    name="${prefix}_Mecanum_roller_joint_2"
     type="continuous">
     <origin
@@ -141,12 +147,12 @@
       rpy="1.6775 -0.19406 -0.76608" />
     <parent
-      link="base_link" />
-    <child
-      link="Mecanum_roller_link_2" />
-    <axis
-      xyz="1 0 0" />
-  </joint>
-  <link
-    name="Mecanum_roller_link_3">
+      link="${prefix}_link" />
+    <child
+      link="${prefix}_Mecanum_roller_link_2" />
+    <axis
+      xyz="1 0 0" />
+  </joint>
+  <link
+    name="${prefix}_Mecanum_roller_link_3">
     <inertial>
       <origin
@@ -188,5 +194,5 @@
   </link>
   <joint
-    name="Mecanum_roller_joint_3"
+    name="${prefix}_Mecanum_roller_joint_3"
     type="continuous">
     <origin
@@ -194,12 +200,12 @@
       rpy="1.4846 0.29377 -0.73958" />
     <parent
-      link="base_link" />
-    <child
-      link="Mecanum_roller_link_3" />
-    <axis
-      xyz="1 0 0" />
-  </joint>
-  <link
-    name="Mecanum_roller_link_4">
+      link="${prefix}_link" />
+    <child
+      link="${prefix}_Mecanum_roller_link_3" />
+    <axis
+      xyz="1 0 0" />
+  </joint>
+  <link
+    name="${prefix}_Mecanum_roller_link_4">
     <inertial>
       <origin
@@ -241,5 +247,5 @@
   </link>
   <joint
-    name="Mecanum_roller_joint_4"
+    name="${prefix}_Mecanum_roller_joint_4"
     type="continuous">
     <origin
@@ -247,12 +253,12 @@
       rpy="1.4497 0.68992 -0.41086" />
     <parent
-      link="base_link" />
-    <child
-      link="Mecanum_roller_link_4" />
-    <axis
-      xyz="1 0 0" />
-  </joint>
-  <link
-    name="Mecanum_roller_link_5">
+      link="${prefix}_link" />
+    <child
+      link="${prefix}_Mecanum_roller_link_4" />
+    <axis
+      xyz="1 0 0" />
+  </joint>
+  <link
+    name="${prefix}_Mecanum_roller_link_5">
     <inertial>
       <origin
@@ -294,5 +300,5 @@
   </link>
   <joint
-    name="Mecanum_roller_joint_5"
+    name="${prefix}_Mecanum_roller_joint_5"
     type="continuous">
     <origin
@@ -300,12 +306,12 @@
       rpy="1.6948 0.7554 0.24013" />
     <parent
-      link="base_link" />
-    <child
-      link="Mecanum_roller_link_5" />
-    <axis
-      xyz="1 0 0" />
-  </joint>
-  <link
-    name="Mecanum_roller_link_6">
+      link="${prefix}_link" />
+    <child
+      link="${prefix}_Mecanum_roller_link_5" />
+    <axis
+      xyz="1 0 0" />
+  </joint>
+  <link
+    name="${prefix}_Mecanum_roller_link_6">
     <inertial>
       <origin
@@ -347,5 +353,5 @@
   </link>
   <joint
-    name="Mecanum_roller_joint_6"
+    name="${prefix}_Mecanum_roller_joint_6"
     type="continuous">
     <origin
@@ -353,12 +359,12 @@
       rpy="1.7524 0.42673 0.68129" />
     <parent
-      link="base_link" />
-    <child
-      link="Mecanum_roller_link_6" />
-    <axis
-      xyz="1 0 0" />
-  </joint>
-  <link
-    name="Mecanum_roller_link_7">
+      link="${prefix}_link" />
+    <child
+      link="${prefix}_Mecanum_roller_link_6" />
+    <axis
+      xyz="1 0 0" />
+  </joint>
+  <link
+    name="${prefix}_Mecanum_roller_link_7">
     <inertial>
       <origin
@@ -400,5 +406,5 @@
   </link>
   <joint
-    name="Mecanum_roller_joint_7"
+    name="${prefix}_Mecanum_roller_joint_7"
     type="continuous">
     <origin
@@ -406,12 +412,12 @@
       rpy="2.5112 -0.051481 0.78407" />
     <parent
-      link="base_link" />
-    <child
-      link="Mecanum_roller_link_7" />
-    <axis
-      xyz="1 0 0" />
-  </joint>
-  <link
-    name="Mecanum_roller_link_8">
+      link="${prefix}_link" />
+    <child
+      link="${prefix}_Mecanum_roller_link_7" />
+    <axis
+      xyz="1 0 0" />
+  </joint>
+  <link
+    name="${prefix}_Mecanum_roller_link_8">
     <inertial>
       <origin
@@ -453,5 +459,5 @@
   </link>
   <joint
-    name="Mecanum_roller_joint_8"
+    name="${prefix}_Mecanum_roller_joint_8"
     type="continuous">
     <origin
@@ -459,12 +465,12 @@
       rpy="-1.7252 -0.51523 0.6222" />
     <parent
-      link="base_link" />
-    <child
-      link="Mecanum_roller_link_8" />
-    <axis
-      xyz="1 0 0" />
-  </joint>
-  <link
-    name="Mecanum_roller_link_9">
+      link="${prefix}_link" />
+    <child
+      link="${prefix}_Mecanum_roller_link_8" />
+    <axis
+      xyz="1 0 0" />
+  </joint>
+  <link
+    name="${prefix}_Mecanum_roller_link_9">
     <inertial>
       <origin
@@ -506,5 +512,5 @@
   </link>
   <joint
-    name="Mecanum_roller_joint_9"
+    name="${prefix}_Mecanum_roller_joint_9"
     type="continuous">
     <origin
@@ -512,94 +518,10 @@
       rpy="1.5575 -0.78024 0.10117" />
     <parent
-      link="base_link" />
-    <child
-      link="Mecanum_roller_link_9" />
-    <axis
-      xyz="1 0 0" />
-  </joint>
-    <ros2_control name="gazeboSimSystem" type="system">
-		<hardware>
-			<plugin>gazebo_ros2_control/GazeboSystem</plugin>
-		</hardware>
-		<joint name="Mecanum_roller_joint_1">
-			<command_interface name="velocity">
-				<param name="min">-100</param>
-				<param name="max">100</param>
-			</command_interface>
-			<state_interface name="position"/>
-			<state_interface name="velocity"/>
-		</joint>
-		<joint name="Mecanum_roller_joint_2">
-			<command_interface name="velocity">
-				<param name="min">-100</param>
-				<param name="max">100</param>
-			</command_interface>
-			<state_interface name="position"/>
-			<state_interface name="velocity"/>
-		</joint>
-    		<joint name="Mecanum_roller_joint_3">
-			<command_interface name="velocity">
-				<param name="min">-100</param>
-				<param name="max">100</param>
-			</command_interface>
-			<state_interface name="position"/>
-			<state_interface name="velocity"/>
-		</joint>
-    		<joint name="Mecanum_roller_joint_4">
-			<command_interface name="velocity">
-				<param name="min">-100</param>
-				<param name="max">100</param>
-			</command_interface>
-			<state_interface name="position"/>
-			<state_interface name="velocity"/>
-		</joint>
-    		<joint name="Mecanum_roller_joint_5">
-			<command_interface name="velocity">
-				<param name="min">-100</param>
-				<param name="max">100</param>
-			</command_interface>
-			<state_interface name="position"/>
-			<state_interface name="velocity"/>
-		</joint>
-    		<joint name="Mecanum_roller_joint_6">
-			<command_interface name="velocity">
-				<param name="min">-100</param>
-				<param name="max">100</param>
-			</command_interface>
-			<state_interface name="position"/>
-			<state_interface name="velocity"/>
-		</joint>
-    		<joint name="Mecanum_roller_joint_7">
-			<command_interface name="velocity">
-				<param name="min">-100</param>
-				<param name="max">100</param>
-			</command_interface>
-			<state_interface name="position"/>
-			<state_interface name="velocity"/>
-		</joint>
-    		<joint name="Mecanum_roller_joint_8">
-			<command_interface name="velocity">
-				<param name="min">-100</param>
-				<param name="max">100</param>
-			</command_interface>
-			<state_interface name="position"/>
-			<state_interface name="velocity"/>
-		</joint>
-    		<joint name="Mecanum_roller_joint_9">
-			<command_interface name="velocity">
-				<param name="min">-100</param>
-				<param name="max">100</param>
-			</command_interface>
-			<state_interface name="position"/>
-			<state_interface name="velocity"/>
-		</joint>
-	</ros2_control>
-  	<gazebo>
-		<plugin filename="libgazebo_ros2_control.so" name="gazebo_ros2_control">
-			<parameters>$(find icarus_pi)/config/controllers.yaml</parameters>
-			<robot_param>robot_description</robot_param>
-			<robot_param_node>robot_state_publisher</robot_param_node>
-			<controller_manager_name>icarus_controller_manager</controller_manager_name>
-		</plugin>
-	</gazebo>
+      link="${prefix}_link" />
+    <child
+      link="${prefix}_Mecanum_roller_link_9" />
+    <axis
+      xyz="1 0 0" />
+  </joint>
+  </xacro:macro>
 </robot>

File: src/icarus_pi/description/Mecanum-Right.urdf.xacro (robot description, xacro)
@@ -1,10 +1,7 @@
 <?xml version="1.0" encoding="utf-8"?>
-<!-- This URDF was automatically created by SolidWorks to URDF Exporter! Originally created by Stephen Brawner (brawner@gmail.com)
-     Commit Version: 1.6.0-4-g7f85cfe  Build Version: 1.6.7995.38578
-     For more information, please see http://wiki.ros.org/sw_urdf_exporter -->
-<robot
-  name="Mecanum-Right">
-  <link
-    name="Right_Base_Link">
+<robot xmlns:xacro="http://www.ros.org/wiki/xacro" >
+  <xacro:macro name="MecanumR" params="prefix x_reflect y_reflect">
+  <link
+    name="${prefix}_link">
     <inertial>
       <origin
@@ -45,6 +42,12 @@
     </collision>
   </link>
-  <link
-    name="Mecanum_Roller_Link1">
+  <joint name="${prefix}_joint" type="continuous">
+		<parent link="base_link"/>
+		<child link="${prefix}_link"/>
+		<origin xyz="${x_reflect*wheel_xoff} ${y_reflect*(chassis_width/2 + wheel_ygap)} ${-wheel_zoff}" rpy="0 0 0"/>
+    <axis xyz="0 0 1"/>
+	</joint>
+  <link
+    name="${prefix}_Mecanum_Roller_Link1">
     <inertial>
       <origin
@@ -86,5 +89,5 @@
   </link>
   <joint
-    name="Mecanum_Roller_Joint_1"
+    name="${prefix}_Mecanum_Roller_Joint_1"
     type="continuous">
     <origin
@@ -92,12 +95,12 @@
       rpy="-1.36068806852681 0.491674447872911 -2.73783219400761" />
     <parent
-      link="Right_Base_Link" />
-    <child
-      link="Mecanum_Roller_Link1" />
-    <axis
-      xyz="1 0 0" />
-  </joint>
-  <link
-    name="Mecanum_Roller_Link2">
+      link="${prefix}_link" />
+    <child
+      link="${prefix}_Mecanum_Roller_Link1" />
+    <axis
+      xyz="1 0 0" />
+  </joint>
+  <link
+    name="${prefix}_Mecanum_Roller_Link2">
     <inertial>
       <origin
@@ -139,5 +142,5 @@
   </link>
   <joint
-    name="Mecanum_Roller_Joint_2"
+    name="${prefix}_Mecanum_Roller_Joint_2"
     type="continuous">
     <origin
@@ -145,12 +148,12 @@
       rpy="1.93542758330994 -0.0214038442701011 0.265392618762669" />
     <parent
-      link="Right_Base_Link" />
-    <child
-      link="Mecanum_Roller_Link2" />
-    <axis
-      xyz="1 0 0" />
-  </joint>
-  <link
-    name="Mecanum_Roller_Link3">
+      link="${prefix}_link" />
+    <child
+      link="${prefix}_Mecanum_Roller_Link2" />
+    <axis
+      xyz="1 0 0" />
+  </joint>
+  <link
+    name="${prefix}_Mecanum_Roller_Link3">
     <inertial>
       <origin
@@ -192,5 +195,5 @@
   </link>
   <joint
-    name="Mecanum_Roller_Joint_3"
+    name="${prefix}_Mecanum_Roller_Joint_3"
     type="continuous">
     <origin
@@ -198,12 +201,12 @@
       rpy="-1.45997240902279 -0.325004631734415 3.05656776956051" />
     <parent
-      link="Right_Base_Link" />
-    <child
-      link="Mecanum_Roller_Link3" />
-    <axis
-      xyz="1 0 0" />
-  </joint>
-  <link
-    name="Mecanum_Roller_Link4">
+      link="${prefix}_link" />
+    <child
+      link="${prefix}_Mecanum_Roller_Link3" />
+    <axis
+      xyz="1 0 0" />
+  </joint>
+  <link
+    name="${prefix}_Mecanum_Roller_Link4">
     <inertial>
       <origin
@@ -245,5 +248,5 @@
   </link>
   <joint
-    name="Mecanum_Roller_Joint_4"
+    name="${prefix}_Mecanum_Roller_Joint_4"
     type="continuous">
     <origin
@@ -251,12 +254,12 @@
       rpy="-1.23509707840396 0.401303910502291 -0.602154738197085" />
     <parent
-      link="Right_Base_Link" />
-    <child
-      link="Mecanum_Roller_Link4" />
-    <axis
-      xyz="1 0 0" />
-  </joint>
-  <link
-    name="Mecanum_Roller_Link5">
+      link="${prefix}_link" />
+    <child
+      link="${prefix}_Mecanum_Roller_Link4" />
+    <axis
+      xyz="1 0 0" />
+  </joint>
+  <link
+    name="${prefix}_Mecanum_Roller_Link5">
     <inertial>
       <origin
@@ -298,5 +301,5 @@
   </link>
   <joint
-    name="Mecanum_Roller_Joint_5"
+    name="${prefix}_Mecanum_Roller_Joint_5"
     type="continuous">
     <origin
@@ -304,12 +307,12 @@
       rpy="1.01038415879456 0.159830081855345 -1.04575970415485" />
     <parent
-      link="Right_Base_Link" />
-    <child
-      link="Mecanum_Roller_Link5" />
-    <axis
-      xyz="1 0 0" />
-  </joint>
-  <link
-    name="Mecanum_Roller_Link6">
+      link="${prefix}_link" />
+    <child
+      link="${prefix}_Mecanum_Roller_Link5" />
+    <axis
+      xyz="1 0 0" />
+  </joint>
+  <link
+    name="${prefix}_Mecanum_Roller_Link6">
     <inertial>
       <origin
@@ -351,5 +354,5 @@
   </link>
   <joint
-    name="Mecanum_Roller_Joint_6"
+    name="${prefix}_Mecanum_Roller_Joint_6"
     type="continuous">
     <origin
@@ -357,12 +360,12 @@
       rpy="-1.00833638122774 -0.270056335980709 -1.28003202448786" />
     <parent
-      link="Right_Base_Link" />
-    <child
-      link="Mecanum_Roller_Link6" />
-    <axis
-      xyz="1 0 0" />
-  </joint>
-  <link
-    name="Mecanum_Roller_Link7">
+      link="${prefix}_link" />
+    <child
+      link="${prefix}_Mecanum_Roller_Link6" />
+    <axis
+      xyz="1 0 0" />
+  </joint>
+  <link
+    name="${prefix}_Mecanum_Roller_Link7">
     <inertial>
       <origin
@@ -404,5 +407,5 @@
   </link>
   <joint
-    name="Mecanum_Roller_Joint_7"
+    name="${prefix}_Mecanum_Roller_Joint_7"
     type="continuous">
     <origin
@@ -410,12 +413,12 @@
       rpy="0.755293558147071 0.758576984655219 1.85745610617137" />
     <parent
-      link="Right_Base_Link" />
-    <child
-      link="Mecanum_Roller_Link7" />
-    <axis
-      xyz="1 0 0" />
-  </joint>
-  <link
-    name="Mecanum_Roller_Link8">
+      link="${prefix}_link" />
+    <child
+      link="${prefix}_Mecanum_Roller_Link7" />
+    <axis
+      xyz="1 0 0" />
+  </joint>
+  <link
+    name="${prefix}_Mecanum_Roller_Link8">
     <inertial>
       <origin
@@ -457,5 +460,5 @@
   </link>
   <joint
-    name="Mecanum_Roller_Joint_8"
+    name="${prefix}_Mecanum_Roller_Joint_8"
     type="continuous">
     <origin
@@ -463,12 +466,12 @@
       rpy="2.95463100680286 -1.13639269714102 -0.725426795925048" />
     <parent
-      link="Right_Base_Link" />
-    <child
-      link="Mecanum_Roller_Link8" />
-    <axis
-      xyz="1 0 0" />
-  </joint>
-  <link
-    name="Mecanum_Roller_Link9">
+      link="${prefix}_link" />
+    <child
+      link="${prefix}_Mecanum_Roller_Link8" />
+    <axis
+      xyz="1 0 0" />
+  </joint>
+  <link
+    name="${prefix}_Mecanum_Roller_Link9">
     <inertial>
       <origin
@@ -510,5 +513,5 @@
   </link>
   <joint
-    name="Mecanum_Roller_Joint_9"
+    name="${prefix}_Mecanum_Roller_Joint_9"
     type="continuous">
     <origin
@@ -516,94 +519,10 @@
       rpy="0.326455693966909 0.964739218565908 -2.90683123969866" />
     <parent
-      link="Right_Base_Link" />
-    <child
-      link="Mecanum_Roller_Link9" />
-    <axis
-      xyz="1 0 0" />
-  </joint>
-    <ros2_control name="gazeboSimSystem" type="system">
-		<hardware>
-			<plugin>gazebo_ros2_control/GazeboSystem</plugin>
-		</hardware>
-		<joint name="Mecanum_roller_joint_1">
-			<command_interface name="velocity">
-				<param name="min">-100</param>
-				<param name="max">100</param>
-			</command_interface>
-			<state_interface name="position"/>
-			<state_interface name="velocity"/>
-		</joint>
-		<joint name="Mecanum_roller_joint_2">
-			<command_interface name="velocity">
-				<param name="min">-100</param>
-				<param name="max">100</param>
-			</command_interface>
-			<state_interface name="position"/>
-			<state_interface name="velocity"/>
-		</joint>
-    		<joint name="Mecanum_roller_joint_3">
-			<command_interface name="velocity">
-				<param name="min">-100</param>
-				<param name="max">100</param>
-			</command_interface>
-			<state_interface name="position"/>
-			<state_interface name="velocity"/>
-		</joint>
-    		<joint name="Mecanum_roller_joint_4">
-			<command_interface name="velocity">
-				<param name="min">-100</param>
-				<param name="max">100</param>
-			</command_interface>
-			<state_interface name="position"/>
-			<state_interface name="velocity"/>
-		</joint>
-    		<joint name="Mecanum_roller_joint_5">
-			<command_interface name="velocity">
-				<param name="min">-100</param>
-				<param name="max">100</param>
-			</command_interface>
-			<state_interface name="position"/>
-			<state_interface name="velocity"/>
-		</joint>
-    		<joint name="Mecanum_roller_joint_6">
-			<command_interface name="velocity">
-				<param name="min">-100</param>
-				<param name="max">100</param>
-			</command_interface>
-			<state_interface name="position"/>
-			<state_interface name="velocity"/>
-		</joint>
-    		<joint name="Mecanum_roller_joint_7">
-			<command_interface name="velocity">
-				<param name="min">-100</param>
-				<param name="max">100</param>
-			</command_interface>
-			<state_interface name="position"/>
-			<state_interface name="velocity"/>
-		</joint>
-    		<joint name="Mecanum_roller_joint_8">
-			<command_interface name="velocity">
-				<param name="min">-100</param>
-				<param name="max">100</param>
-			</command_interface>
-			<state_interface name="position"/>
-			<state_interface name="velocity"/>
-		</joint>
-    		<joint name="Mecanum_roller_joint_9">
-			<command_interface name="velocity">
-				<param name="min">-100</param>
-				<param name="max">100</param>
-			</command_interface>
-			<state_interface name="position"/>
-			<state_interface name="velocity"/>
-		</joint>
-	</ros2_control>
-  	<gazebo>
-		<plugin filename="libgazebo_ros2_control.so" name="gazebo_ros2_control">
-			<parameters>$(find icarus_pi)/config/controllers.yaml</parameters>
-			<robot_param>robot_description</robot_param>
-			<robot_param_node>robot_state_publisher</robot_param_node>
-			<controller_manager_name>icarus_controller_manager</controller_manager_name>
-		</plugin>
-	</gazebo>
+      link="${prefix}_link" />
+    <child
+      link="${prefix}_Mecanum_Roller_Link9" />
+    <axis
+      xyz="1 0 0" />
+  </joint>
+  </xacro:macro>
 </robot>

File: src/icarus_pi/description/lidar.xacro (robot description, xacro)
@@ -15,5 +15,5 @@
 		</collision>
 		<visual>
-			<origin xyz = "${-chassis_length/2 + 2*lidar_radius} 0 ${chassis_height/2}" rpy="0 0 0"/>
+			<origin xyz = "${-chassis_length/2 + 2*lidar_radius} 0 ${chassis_height/4}" rpy="0 0 0"/>
 			<geometry>
 				<cylinder radius="${lidar_radius}" length=".06"/>

File: src/icarus_pi/description/robot_core.xacro (robot description, xacro)
@@ -41,34 +41,10 @@
         <material>Gazebo/White</material>
     </gazebo>
-    <!-- wheels -->
-	<xacro:macro name="wheel" params="prefix x_reflect y_reflect">
-        <joint name="${prefix}_joint" type="continuous">
-            <parent link="base_link"/>
-            <child link="${prefix}_link"/>
-            <origin xyz="${x_reflect*wheel_xoff} ${y_reflect*(chassis_width/2 + wheel_ygap)} ${-wheel_zoff}" rpy="-${pi/2} 0 0"/>
-            <axis xyz="0 0 1"/>
-        </joint>
-        <link name ="${prefix}_link">
-			<collision>
-				<geometry>
-					<cylinder radius="${wheel_radius}" length="${wheel_width}"/>
-				</geometry>
-			</collision>
-            <xacro:inertial_cylinder mass="${wheel_mass}" length="${wheel_width}" radius="${wheel_radius}">
-                <origin xyz="0 0 0" rpy="0 0 0"/>
-            </xacro:inertial_cylinder>
-			<visual>
-				<geometry>
-					<cylinder radius="${wheel_radius}" length="${wheel_width}"/>
-				</geometry>
-				<material name="Gray">
-					<color rgba="0.5 0.5 0.5 1.0"/>
-				</material>
-			</visual>
-	    </link>
-	</xacro:macro>
-	<xacro:wheel prefix="frontLeft" x_reflect="-1" y_reflect="-1"/>
-	<xacro:wheel prefix="frontRight" x_reflect="-1" y_reflect="1"/>
-	<xacro:wheel prefix="backLeft" x_reflect="1" y_reflect="-1"/>
-	<xacro:wheel prefix="backRight" x_reflect="1" y_reflect="1"/>
+     <!-- CHASSIS LINK -->
+    <xacro:include filename="Mecanum-Left.urdf.xacro"/>
+    <xacro:MecanumL prefix="frontRight" x_reflect="-1" y_reflect="1"/>
+    <xacro:MecanumL prefix="backLeft" x_reflect="1" y_reflect="-1"/>
+    <xacro:include filename="Mecanum-Right.urdf.xacro"/>
+    <xacro:MecanumR prefix="frontLeft" x_reflect="-1" y_reflect="-1"/>
+    <xacro:MecanumR prefix="backRight" x_reflect="1" y_reflect="1"/>
 </robot>
