Commit message: Fixed urdf description to right wheel
Need to edit left wheel URDF to revolve around center axis

File: src/icarus_pi/description/Mecanum-Left.urdf.xacro (robot description, xacro)
@@ -1,10 +1,10 @@
 <?xml version="1.0"?>
 <robot xmlns:xacro="http://www.ros.org/wiki/xacro" >
-  <xacro:macro name="Mecanum" params="prefix x_reflect y_reflect r_reflect">
+  <xacro:macro name="Mecanum-Left" params="prefix x_reflect y_reflect r_reflect">
   <link
     name="${prefix}_link">
     <inertial>
       <origin
-        xyz="0.011813 0.0074643 0.015042"
+        xyz="0 0 0"
         rpy="0 0 0" />
       <mass
@@ -49,5 +49,5 @@
         </joint>
   <link
-    name="Mecanum_roller_link_1">
+    name="${prefix}_Mecanum_roller_link_1">
     <inertial>
       <origin
@@ -308,5 +308,5 @@
       link="${prefix}_link" />
     <child
-      link="${prefix}_Mecanum_roller_joint_5" />
+      link="${prefix}_Mecanum_roller_link_5" />
     <axis
       xyz="1 0 0" />
@@ -427,10 +427,10 @@
         value="0.001" />
       <inertia
-        ixx="0"
-        ixy="0"
-        ixz="0"
-        iyy="0"
+        ixx="1.1179E-08"
+        ixy="3.6189E-24"
+        ixz="-4.1359E-25"
+        iyy="3.946E-08"
         iyz="0"
-        izz="0" />
+        izz="3.946E-08" />
     </inertial>
     <visual>
@@ -465,7 +465,7 @@
       rpy="-2.1509048893029 0 -0.78539816339745" />
     <parent
+      link="${prefix}_link" />
+    <child
       link="${prefix}_Mecanum_roller_link_8" />
-    <child
-      link="Mecanum_roller_link_8" />
     <axis
       xyz="1 0 0" />

File: src/icarus_pi/description/Mecanum-Right.urdf.xacro (robot description, xacro)
@@ -6,5 +6,5 @@
       <inertial>
         <origin
-          xyz="1.26236935779668E-18 6.8753657118438E-18 -1.82537623615078E-18"
+          xyz="0 0 0"
           rpy="0 0 0" />
         <mass
@@ -24,5 +24,5 @@
         <geometry>
           <mesh
-            filename="package://Mecanum-8J-Right/meshes/base_link.STL" />
+            filename="file://$(find icarus_pi)/Mesh/Mecanum-8J-Right/meshes/base_link.STL" />
         </geometry>
         <material
@@ -38,8 +38,14 @@
         <geometry>
           <mesh
-            filename="package://Mecanum-8J-Right/meshes/base_link.STL" />
-        </geometry>
-      </collision>
-    </link>
+            filename="file://$(find icarus_pi)/Mesh/Mecanum-8J-Right/meshes/base_link.STL" />
+        </geometry>
+      </collision>
+  </link>
+    <joint name="${prefix}_joint" type="continuous">
+              <parent link="base_link"/>
+              <child link="${prefix}_link"/>
+              <origin xyz="${x_reflect*wheel_xoff} ${y_reflect*(chassis_width/2 + wheel_ygap)} ${-wheel_zoff}" rpy="0 ${r_reflect} ${r_reflect}"/>
+    <axis xyz="0 0 1"/>
+        </joint>
     <link
       name="${prefix}_Mecanum_roller_link_1">
@@ -64,25 +70,24 @@
         <geometry>
           <mesh
-            filename="package://Mecanum-8J-Right/meshes/Mecanum_roller_link_1.STL" />
-        </geometry>
-        <material
-          name="">
-          <color
-            rgba="0.69804 0.69804 0.69804 1" />
-        </material>
-      </visual>
-      <collision>
-        <origin
-          xyz="0 0 0"
-          rpy="0 0 0" />
-        <geometry>
-          <mesh
-            filename="package://Mecanum-8J-Right/meshes/Mecanum_roller_link_1.STL" />
-        </geometry>
-      </collision>
-    </link>
-    <joint
-      name="${prefix}_Mecanum_roller_joint_1"
-      type="continuous">
+            filename="file://$(find icarus_pi)/Mesh/Mecanum-8J-Right/meshes/Mecanum_roller_link_1.STL" />
+        </geometry>
+        <material
+          name="">
+          <color
+            rgba="0.69804 0.69804 0.69804 1" />
+        </material>
+      </visual>
+      <collision>
+        <origin
+          xyz="0 0 0"
+          rpy="0 0 0" />
+        <geometry>
+          <mesh
+            filename="file://$(find icarus_pi)/Mesh/Mecanum-8J-Right/meshes/Mecanum_roller_link_1.STL" />
+        </geometry>
+      </collision>
+    </link>
+    <joint
+      name="${prefix}_Mecanum_roller_joint_1" type="continuous">
       <origin
         xyz="0.014612 -0.0091675 0"
@@ -117,19 +122,19 @@
         <geometry>
           <mesh
-            filename="package://Mecanum-8J-Right/meshes/Mecanum_roller_link_3.STL" />
-        </geometry>
-        <material
-          name="">
-          <color
-            rgba="0.69804 0.69804 0.69804 1" />
-        </material>
-      </visual>
-      <collision>
-        <origin
-          xyz="0 0 0"
-          rpy="0 0 0" />
-        <geometry>
-          <mesh
-            filename="package://Mecanum-8J-Right/meshes/Mecanum_roller_link_3.STL" />
+            filename="file://$(find icarus_pi)/Mesh/Mecanum-8J-Right/meshes/Mecanum_roller_link_3.STL" />
+        </geometry>
+        <material
+          name="">
+          <color
+            rgba="0.69804 0.69804 0.69804 1" />
+        </material>
+      </visual>
+      <collision>
+        <origin
+          xyz="0 0 0"
+          rpy="0 0 0" />
+        <geometry>
+          <mesh
+            filename="file://$(find icarus_pi)/Mesh/Mecanum-8J-Right/meshes/Mecanum_roller_link_3.STL" />
         </geometry>
       </collision>
@@ -170,19 +175,19 @@
         <geometry>
           <mesh
-            filename="package://Mecanum-8J-Right/meshes/Mecanum_roller_link_4.STL" />
-        </geometry>
-        <material
-          name="">
-          <color
-            rgba="0.69804 0.69804 0.69804 1" />
-        </material>
-      </visual>
-      <collision>
-        <origin
-          xyz="0 0 0"
-          rpy="0 0 0" />
-        <geometry>
-          <mesh
-            filename="package://Mecanum-8J-Right/meshes/Mecanum_roller_link_4.STL" />
+            filename="file://$(find icarus_pi)/Mesh/Mecanum-8J-Right/meshes/Mecanum_roller_link_4.STL" />
+        </geometry>
+        <material
+          name="">
+          <color
+            rgba="0.69804 0.69804 0.69804 1" />
+        </material>
+      </visual>
+      <collision>
+        <origin
+          xyz="0 0 0"
+          rpy="0 0 0" />
+        <geometry>
+          <mesh
+            filename="file://$(find icarus_pi)/Mesh/Mecanum-8J-Right/meshes/Mecanum_roller_link_4.STL" />
         </geometry>
       </collision>
@@ -223,19 +228,19 @@
         <geometry>
           <mesh
-            filename="package://Mecanum-8J-Right/meshes/Mecanum_roller_link_5.STL" />
-        </geometry>
-        <material
-          name="">
-          <color
-            rgba="0.69804 0.69804 0.69804 1" />
-        </material>
-      </visual>
-      <collision>
-        <origin
-          xyz="0 0 0"
-          rpy="0 0 0" />
-        <geometry>
-          <mesh
-            filename="package://Mecanum-8J-Right/meshes/Mecanum_roller_link_5.STL" />
+            filename="file://$(find icarus_pi)/Mesh/Mecanum-8J-Right/meshes/Mecanum_roller_link_5.STL" />
+        </geometry>
+        <material
+          name="">
+          <color
+            rgba="0.69804 0.69804 0.69804 1" />
+        </material>
+      </visual>
+      <collision>
+        <origin
+          xyz="0 0 0"
+          rpy="0 0 0" />
+        <geometry>
+          <mesh
+            filename="file://$(find icarus_pi)/Mesh/Mecanum-8J-Right/meshes/Mecanum_roller_link_5.STL" />
         </geometry>
       </collision>
@@ -276,19 +281,19 @@
         <geometry>
           <mesh
-            filename="package://Mecanum-8J-Right/meshes/Mecanum_roller_link_6.STL" />
-        </geometry>
-        <material
-          name="">
-          <color
-            rgba="0.69804 0.69804 0.69804 1" />
-        </material>
-      </visual>
-      <collision>
-        <origin
-          xyz="0 0 0"
-          rpy="0 0 0" />
-        <geometry>
-          <mesh
-            filename="package://Mecanum-8J-Right/meshes/Mecanum_roller_link_6.STL" />
+            filename="file://$(find icarus_pi)/Mesh/Mecanum-8J-Right/meshes/Mecanum_roller_link_6.STL" />
+        </geometry>
+        <material
+          name="">
+          <color
+            rgba="0.69804 0.69804 0.69804 1" />
+        </material>
+      </visual>
+      <collision>
+        <origin
+          xyz="0 0 0"
+          rpy="0 0 0" />
+        <geometry>
+          <mesh
+            filename="file://$(find icarus_pi)/Mesh/Mecanum-8J-Right/meshes/Mecanum_roller_link_6.STL" />
         </geometry>
       </collision>
@@ -329,19 +334,19 @@
         <geometry>
           <mesh
-            filename="package://Mecanum-8J-Right/meshes/Mecanum_roller_link_7.STL" />
-        </geometry>
-        <material
-          name="">
-          <color
-            rgba="0.69804 0.69804 0.69804 1" />
-        </material>
-      </visual>
-      <collision>
-        <origin
-          xyz="0 0 0"
-          rpy="0 0 0" />
-        <geometry>
-          <mesh
-            filename="package://Mecanum-8J-Right/meshes/Mecanum_roller_link_7.STL" />
+            filename="file://$(find icarus_pi)/Mesh/Mecanum-8J-Right/meshes/Mecanum_roller_link_7.STL" />
+        </geometry>
+        <material
+          name="">
+          <color
+            rgba="0.69804 0.69804 0.69804 1" />
+        </material>
+      </visual>
+      <collision>
+        <origin
+          xyz="0 0 0"
+          rpy="0 0 0" />
+        <geometry>
+          <mesh
+            filename="file://$(find icarus_pi)/Mesh/Mecanum-8J-Right/meshes/Mecanum_roller_link_7.STL" />
         </geometry>
       </collision>
@@ -382,19 +387,19 @@
         <geometry>
           <mesh
-            filename="package://Mecanum-8J-Right/meshes/Mecanum_roller_link_8.STL" />
-        </geometry>
-        <material
-          name="">
-          <color
-            rgba="0.69804 0.69804 0.69804 1" />
-        </material>
-      </visual>
-      <collision>
-        <origin
-          xyz="0 0 0"
-          rpy="0 0 0" />
-        <geometry>
-          <mesh
-            filename="package://Mecanum-8J-Right/meshes/Mecanum_roller_link_8.STL" />
+            filename="file://$(find icarus_pi)/Mesh/Mecanum-8J-Right/meshes/Mecanum_roller_link_8.STL" />
+        </geometry>
+        <material
+          name="">
+          <color
+            rgba="0.69804 0.69804 0.69804 1" />
+        </material>
+      </visual>
+      <collision>
+        <origin
+          xyz="0 0 0"
+          rpy="0 0 0" />
+        <geometry>
+          <mesh
+            filename="file://$(find icarus_pi)/Mesh/Mecanum-8J-Right/meshes/Mecanum_roller_link_8.STL" />
         </geometry>
       </collision>
@@ -435,19 +440,19 @@
         <geometry>
           <mesh
-            filename="package://Mecanum-8J-Right/meshes/Mecanum_roller_link_2.STL" />
-        </geometry>
-        <material
-          name="">
-          <color
-            rgba="0.69804 0.69804 0.69804 1" />
-        </material>
-      </visual>
-      <collision>
-        <origin
-          xyz="0 0 0"
-          rpy="0 0 0" />
-        <geometry>
-          <mesh
-            filename="package://Mecanum-8J-Right/meshes/Mecanum_roller_link_2.STL" />
+            filename="file://$(find icarus_pi)/Mesh/Mecanum-8J-Right/meshes/Mecanum_roller_link_2.STL" />
+        </geometry>
+        <material
+          name="">
+          <color
+            rgba="0.69804 0.69804 0.69804 1" />
+        </material>
+      </visual>
+      <collision>
+        <origin
+          xyz="0 0 0"
+          rpy="0 0 0" />
+        <geometry>
+          <mesh
+            filename="file://$(find icarus_pi)/Mesh/Mecanum-8J-Right/meshes/Mecanum_roller_link_2.STL" />
         </geometry>
       </collision>

File: src/icarus_pi/description/robot_core.xacro (robot description, xacro)
@@ -44,7 +44,7 @@
     <xacro:include filename="Mecanum-Left.urdf.xacro"/>
     <xacro:include filename="Mecanum-Right.urdf.xacro"/>
-    <xacro:Mecanum prefix="frontRight" x_reflect="-1" y_reflect="1" r_reflect="${pi/2}"/>
-    <xacro:Mecanum prefix="backLeft" x_reflect="1" y_reflect="-1" r_reflect="${pi/2}"/>
-    <xacro:Mecanum prefix="frontLeft" x_reflect="-1" y_reflect="-1" r_reflect="${pi/2}"/>
-    <xacro:Mecanum prefix="backRight" x_reflect="1" y_reflect="1" r_reflect="${pi/2}"/>
+    <xacro:Mecanum-Right prefix="frontRight" x_reflect="-1" y_reflect="1" r_reflect="${pi/2}"/>
+    <xacro:Mecanum-Left prefix="backLeft" x_reflect="1" y_reflect="-1" r_reflect="${pi/2}"/>
+    <xacro:Mecanum-Left prefix="frontLeft" x_reflect="-1" y_reflect="-1" r_reflect="${pi/2}"/>
+    <xacro:Mecanum-Right prefix="backRight" x_reflect="1" y_reflect="1" r_reflect="${pi/2}"/>
 </robot>
