Commit message: Added inertial parameters to mecanum urdfs

File: src/icarus_pi/description/Mecanum-8J-Left.urdf.xacro (robot description, xacro)
@@ -1,5 +1,5 @@
 <?xml version="1.0"?>
 <robot xmlns:xacro="http://www.ros.org/wiki/xacro" >
-  <xacro:macro name="Mecanum-Left" params="prefix x_reflect y_reflect r_reflect">
+  <xacro:macro name="Mecanum-Left" params="prefix x_reflect y_reflect r_reflect mass radius length">
     <link
       name="${prefix}_link">
@@ -11,10 +11,10 @@
           value="0.01257" />
         <inertia
-          ixx="1.6068E-06"
-          ixy="-1.346E-21"
-          ixz="-1.6753E-21"
-          iyy="1.1358E-06"
-          iyz="1.5878E-22"
-          izz="1.1358E-06" />
+          ixx="${(1/12) * mass * (3*radius*radius + length*length)}"
+          ixy="0"
+          ixz="0"
+          iyy="${(1/12) * mass * (3*radius*radius + length*length)}"
+          iyz="0"
+          izz="${(1/2) * mass * (radius*radius)}" />
       </inertial>
       <visual>

File: src/icarus_pi/description/Mecanum-Right.urdf.xacro (robot description, xacro)
@@ -1,5 +1,5 @@
 <?xml version="1.0"?>
 <robot xmlns:xacro="http://www.ros.org/wiki/xacro" >
-  <xacro:macro name="Mecanum-Right" params="prefix x_reflect y_reflect r_reflect">
+  <xacro:macro name="Mecanum-Right" params="prefix x_reflect y_reflect r_reflect mass radius length">
     <link
       name="${prefix}_link">
@@ -11,10 +11,10 @@
           value="0.0118270309310726" />
         <inertia
-          ixx="1.05151006190876E-06"
-          ixy="1.716037457491E-21"
-          ixz="5.05880721300189E-23"
-          iyy="1.4398222580115E-06"
-          iyz="-4.33869183207793E-22"
-          izz="1.05151006190876E-06" />
+          ixx="${(1/12) * mass * (3*radius*radius + length*length)}"
+          ixy="0"
+          ixz="0"
+          iyy="${(1/12) * mass * (3*radius*radius + length*length)}"
+          iyz="0"
+          izz="${(1/2) * mass * (radius*radius)}" />
       </inertial>
       <visual>

File: src/icarus_pi/description/robot_core.xacro (robot description, xacro)
@@ -10,5 +10,5 @@
         <parent link="base_link"/>
         <child link="base_footprint"/>
-        <origin xyz="0 0 0" rpy="0 0 0"/>
+        <origin xyz="0 0 1" rpy="0 0 0"/>
     </joint>
     <link name="base_footprint">
@@ -44,7 +44,7 @@
     <xacro:include filename="Mecanum-8J-Left.urdf.xacro"/>
     <xacro:include filename="Mecanum-Right.urdf.xacro"/>
-    <xacro:Mecanum-Right prefix="frontRight" x_reflect="-1" y_reflect="1" r_reflect="${pi/2}"/>
-    <xacro:Mecanum-Right prefix="backLeft" x_reflect="1" y_reflect="-1" r_reflect="${pi/2}"/>
-    <xacro:Mecanum-Left prefix="frontLeft" x_reflect="-1" y_reflect="-1" r_reflect="${pi/2}"/>
-    <xacro:Mecanum-Left prefix="backRight" x_reflect="1" y_reflect="1" r_reflect="${pi/2}"/>
+    <xacro:Mecanum-Right prefix="frontRight" x_reflect="-1" y_reflect="1" r_reflect="${pi/2}" mass="${wheel_mass}" radius="${wheel_radius}" length="${wheel_width}"/>
+    <xacro:Mecanum-Right prefix="backLeft" x_reflect="1" y_reflect="-1" r_reflect="${pi/2}" mass="${wheel_mass}" radius="${wheel_radius}" length="${wheel_width}"/>
+    <xacro:Mecanum-Left prefix="frontLeft" x_reflect="-1" y_reflect="-1" r_reflect="${pi/2}" mass="${wheel_mass}" radius="${wheel_radius}" length="${wheel_width}"/>
+    <xacro:Mecanum-Left prefix="backRight" x_reflect="1" y_reflect="1" r_reflect="${pi/2}" mass="${wheel_mass}" radius="${wheel_radius}" length="${wheel_width}"/>
 </robot>

File: src/icarus_pi/description/robot_dimensions.xacro (robot description, xacro)
@@ -5,5 +5,5 @@
     <xacro:property name="chassis_width" value = ".203"/>
     <xacro:property name="chassis_height" value = ".16"/>
-    <xacro:property name="chassis_mass" value = "10"/>
+    <xacro:property name="chassis_mass" value = "20"/>
     <xacro:property name="wheel_radius" value = ".024"/>
     <xacro:property name="wheel_width" value = ".03"/>
@@ -11,5 +11,5 @@
     <xacro:property name="wheel_ygap" value = ".018"/>
     <xacro:property name="wheel_xoff" value = ".1015"/>
-    <xacro:property name="wheel_mass" value = "1"/>
+    <xacro:property name="wheel_mass" value = ".022"/>
     <xacro:property name="support_height" value = ".203"/>
     <xacro:property name="support_radius" value = ".203"/>
