Commit message: Added gazebo planar plugin to ros2_control.xacro. Modified wheel joints to be fixed in sim and continuous in real world in robot_core.xacro. Cleaned up and added link materials in gazebo_control.xacro, lidar.xacro, and robot_core.xacro.

File: src/icarus_pi/description/gazebo_control.xacro (robot description, xacro)
@@ -1,4 +1,5 @@
 <?xml version="1.0"?>
 <robot xmlns:xacro="http://www.ros.org/wiki/xacro">
+    <!-- :: WARNING :: FILE NOT USED :: -->
     <gazebo>
         <plugin name="diff_drive" filename="libgazebo_ros_diff_drive.so">

File: src/icarus_pi/description/lidar.xacro (robot description, xacro)
@@ -19,6 +19,6 @@
 				<cylinder radius="${lidar_radius}" length=".06"/>
 			</geometry>
-			<material name="Gray">
-				<color rgba="0.5 0.5 0.5 1.0"/>
+			<material name="black">
+				<color rgba="0 0 0 1"/>
 			</material>
 		</visual>
@@ -29,8 +29,9 @@
 		<parent link="chassis"/>
 		<child link="lidar_link"/>
-		<origin xyz="${lidar_radius} 0 ${chassis_height+.03}" rpy="0 0 0"/>
+		<origin xyz="${lidar_radius} 0 ${chassis_height + 0.03}" rpy="0 0 0"/>
 	</joint>
 	<!--adding gazebo plugins to the sim-->
 	<gazebo reference="lidar_link">
+    	<material>Gazebo/Black</material>
 		<sensor name="lidar" type="ray">
 			<always_on>true</always_on>

File: src/icarus_pi/description/robot_core.xacro (robot description, xacro)
@@ -26,5 +26,5 @@
                 <box size="${chassis_length} ${chassis_width} ${chassis_height}"/>
             </geometry>
-            <material name="white"/>
+            <material name="blue"/>
         </visual>
         <collision>
@@ -39,14 +39,24 @@
     </link>
     <gazebo reference="chassis">
-        <material>Gazebo/White</material>
+        <material>Gazebo/Gray</material>
     </gazebo>
     <!-- wheels -->
 	<xacro:macro name="wheel" params="prefix x_reflect y_reflect">
-        <joint name="${prefix}_joint" type="continuous">
-            <parent link="base_link"/>
-            <child link="${prefix}_link"/>
-            <origin xyz="${x_reflect*wheel_xoff} ${y_reflect*(chassis_width/2 + wheel_ygap)} ${-wheel_zoff}" rpy="-${pi/2} 0 0"/>
-            <axis xyz="0 0 1"/>
-        </joint>
+        <xacro:if value="$(arg sim_mode)">
+            <joint name="${prefix}_joint" type="fixed">
+                <parent link="base_link"/>
+                <child link="${prefix}_link"/>
+                <origin xyz="${x_reflect*wheel_xoff} ${y_reflect*(chassis_width/2 + wheel_ygap)} ${-wheel_zoff}" rpy="-${pi/2} 0 0"/>
+                <axis xyz="0 0 1"/>
+            </joint>
+        </xacro:if>
+        <xacro:unless value="$(arg use_ros2_control)">
+            <joint name="${prefix}_joint" type="continuous">
+                <parent link="base_link"/>
+                <child link="${prefix}_link"/>
+                <origin xyz="${x_reflect*wheel_xoff} ${y_reflect*(chassis_width/2 + wheel_ygap)} ${-wheel_zoff}" rpy="-${pi/2} 0 0"/>
+                <axis xyz="0 0 1"/>
+            </joint>
+        </xacro:unless>
         <link name ="${prefix}_link">
 			<collision>
@@ -62,6 +72,6 @@
 					<cylinder radius="${wheel_radius}" length="${wheel_width}"/>
 				</geometry>
-				<material name="Gray">
-					<color rgba="0.5 0.5 0.5 1.0"/>
+				<material name="Yellow">
+					<color rgba="1 1 0 1"/>
 				</material>
 			</visual>
@@ -72,3 +82,15 @@
 	<xacro:wheel prefix="frontRight" x_reflect="1" y_reflect="-1"/>
 	<xacro:wheel prefix="frontLeft" x_reflect="1" y_reflect="1"/>
+    <gazebo reference="backRight_link">
+        <material>Gazebo/ZincYellow</material>
+    </gazebo>
+    <gazebo reference="backLeft_link">
+        <material>Gazebo/ZincYellow</material>
+    </gazebo>
+    <gazebo reference="frontRight_link">
+        <material>Gazebo/ZincYellow</material>
+    </gazebo>
+    <gazebo reference="frontLeft_link">
+        <material>Gazebo/ZincYellow</material>
+    </gazebo>
 </robot>

File: src/icarus_pi/description/ros2_control.xacro (robot description, xacro)
@@ -91,3 +91,13 @@
         </plugin>
     </gazebo>
+    <gazebo>
+      <plugin name="planar_controller" filename="libgazebo_ros_planar_move.so">
+            <command_topic>cmd_vel</command_topic>
+            <odometry_frame>odom</odometry_frame>
+            <odometry_rate>50.0</odometry_rate>
+            <robot_base_frame>base_link</robot_base_frame>
+            <publish_odom>true</publish_odom>
+            <publish_odom_tf>true</publish_odom_tf>
+        </plugin>
+    </gazebo>
 </robot>

Commit message: Split the planar and ros2 control into two seperate descriptions for easy launch

File: src/icarus_pi/description/gazebo_control.xacro (robot description, xacro)
@@ -1,24 +1,12 @@
 <?xml version="1.0"?>
 <robot xmlns:xacro="http://www.ros.org/wiki/xacro">
-    <!-- :: WARNING :: FILE NOT USED :: -->
-    <gazebo>
-        <plugin name="diff_drive" filename="libgazebo_ros_diff_drive.so">
-            <!-- Wheel Information -->
-            <num_wheel_pairs>2</num_wheel_pairs>
-            <left_joint>frontLeft_joint</left_joint>
-            <left_joint>backLeft_joint</left_joint>
-            <right_joint>frontRight_joint</right_joint>
-            <right_joint>backRight_joint</right_joint>
-            <wheel_separation>0.7</wheel_separation>
-            <wheel_diameter>0.024</wheel_diameter>
-            <!-- Limits -->
-            <max_wheel_torque>500</max_wheel_torque>
-            <max_wheel_acceleration>10.0</max_wheel_acceleration>
-            <!-- Output -->
+   <gazebo>
+      <plugin name="planar_controller" filename="libgazebo_ros_planar_move.so">
+            <command_topic>cmd_vel</command_topic>
             <odometry_frame>odom</odometry_frame>
+            <odometry_rate>50.0</odometry_rate>
             <robot_base_frame>base_link</robot_base_frame>
             <publish_odom>true</publish_odom>
             <publish_odom_tf>true</publish_odom_tf>
-            <publish_wheel_tf>true</publish_wheel_tf>
         </plugin>
     </gazebo>

File: src/icarus_pi/description/gazebo_robot_core.xacro (robot description, xacro)
@@ -41,8 +41,8 @@
     <!-- wheels -->
 	<xacro:macro name="wheel" params="prefix x_reflect y_reflect rotate">
-        <joint name="${prefix}_joint" type="continuous">
+        <joint name="${prefix}_joint" type="fixed">
             <parent link="base_link"/>
             <child link="${prefix}_link"/>
-            <origin xyz="${x_reflect*wheel_xoff} ${y_reflect*(chassis_width/2 + wheel_ygap)} ${-wheel_zoff}" rpy="-${pi/2} 0 ${rotate}"/>
+            <origin xyz="${x_reflect*wheel_xoff} ${y_reflect*(chassis_width/2 + wheel_ygap)} ${-wheel_zoff}" rpy="-${pi/2} 0 0"/>
             <axis xyz="0 0 1"/>
         </joint>

File: src/icarus_pi/description/robot.urdf.xacro (robot description, xacro)
@@ -2,6 +2,15 @@
 <robot xmlns:xacro="http://www.ros.org/wiki/xacro"  name="robot">
     <xacro:arg name="use_ros2_control" default="true"/>
-    <xacro:arg name="sim_mode" default="false"/>
-    <xacro:include filename="robot_core.xacro" />
+    <xacro:arg name="sim_mode" default="true"/>
+    <xacro:include filename="robot_dimensions.xacro"/>
+    <xacro:include filename="inertial_macros.xacro"/>
+    <!--Robot Description Choice-->
+    <xacro:if value="$(arg sim_mode)">
+        <xacro:include filename="gazebo_robot_core.xacro" />
+    </xacro:if>
+    <xacro:unless value="$(arg sim_mode)">
+        <xacro:include filename="robot_core.xacro" />
+    </xacro:unless>
+    <!--Controller Choice-->
     <xacro:if value="$(arg use_ros2_control)">
         <xacro:include filename="ros2_control.xacro" />

File: src/icarus_pi/description/ros2_control.xacro (robot description, xacro)
@@ -91,13 +91,3 @@
         </plugin>
     </gazebo>
-    <gazebo>
-      <plugin name="planar_controller" filename="libgazebo_ros_planar_move.so">
-            <command_topic>cmd_vel</command_topic>
-            <odometry_frame>odom</odometry_frame>
-            <odometry_rate>50.0</odometry_rate>
-            <robot_base_frame>base_link</robot_base_frame>
-            <publish_odom>true</publish_odom>
-            <publish_odom_tf>true</publish_odom_tf>
-        </plugin>
-    </gazebo>
 </robot>
