Commit message: - flipped direction of odometry frame so that robot now moves in the positive directions of the odometry frame when given a positive command (same for negative commands) - changed robot dimensions within yaml to be more accurate to real world wheel seperation measurements - edited odometry file to read in and calculate from proper units of measurement - added logger variables to odometry hpp file - rotated wheel urdf to spin in the correct direction

File: src/icarus_pi/description/robot_core.xacro (robot description, xacro)
@@ -18,5 +18,5 @@
         <parent link="base_link"/>
         <child link="chassis"/>
-        <origin xyz="${-wheel_xoff} 0.0 ${-wheel_zoff}"/>
+        <origin xyz="${-wheel_xoff} 0.0 ${-wheel_zoff}" rpy="0 0 0"/>
     </joint>
     <link name="chassis">
@@ -46,5 +46,5 @@
                 <parent link="base_link"/>
                 <child link="${prefix}_link"/>
-                <origin xyz="${x_reflect*wheel_xoff} ${y_reflect*(chassis_width/2 + wheel_ygap)} ${-wheel_zoff}" rpy="-${pi/2} 0 0"/>
+                <origin xyz="${x_reflect*wheel_xoff} ${y_reflect*(chassis_width/2 + wheel_ygap)} ${-wheel_zoff}" rpy="-${pi/2} 0 ${pi}"/>
                 <axis xyz="0 0 1"/>
             </joint>
