Commit message: Fixed Odom twist messages

File: src/icarus_pi/description/lidar.xacro (robot description, xacro)
@@ -1,70 +1,74 @@
 <?xml version="1.0"?>
 <robot xmlns:xacro="http://www.ros.org/wiki/xacro" >
-    <!--lidar intrinsics-->
-	<link name="lidar_link">
-		<inertial>
-			<origin xyz="${-chassis_length/2 + 2*lidar_radius} 0 ${chassis_height/2}" rpy="0 0 0"/>
-			<mass value=".17"/>
-			<inertia ixx="0.001"  ixy="0"  ixz="0" iyy="0.001" iyz="0" izz="0.001"/>
-		</inertial>
-		<collision>
-			<origin xyz="${-chassis_length/2 + 2*lidar_radius} 0 ${chassis_height/2}"/>
-			<geometry>
-				<cylinder radius="${lidar_radius}" length=".06"/>
-			</geometry>
-		</collision>
-		<visual>
-			<origin xyz = "${-chassis_length/2 + 2*lidar_radius} 0 ${chassis_height/2}" rpy="0 0 0"/>
-			<geometry>
-				<cylinder radius="${lidar_radius}" length=".06"/>
-			</geometry>
-			<material name="Gray">
-				<color rgba="0.5 0.5 0.5 1.0"/>
-			</material>
-		</visual>
-	</link>
-	<!--create the joint that the lidar_link will be bound to with the base being the base_link-->
-	<joint name="lidar_joint" type="fixed">
-	<!--^^make joint continuous to mimic spinning lidar?-->
-		<parent link="base_link"/>
-		<child link="lidar_link"/>
-		<origin xyz="${-chassis_length/2 + lidar_radius} 0 ${chassis_height/2+.02}" rpy="0 0 0"/>
-	</joint>
-    <!--adding gazebo plugins to the sim-->
-	<gazebo reference="lidar_link">
-		<sensor name="lidar" type="ray">
-			<always_on>true</always_on>
-			<visualize>true</visualize>
-			<update_rate>5</update_rate>
-			<ray>
-				<scan>
-					<horizontal>
-						<samples>8000</samples>
+	<xacro:unless value="$(arg sim_mode)">
+		<!--lidar intrinsics-->
+		<link name="lidar_link">
+			<inertial>
+				<origin xyz="${-chassis_length/2 + 2*lidar_radius} 0 ${chassis_height/2}" rpy="0 0 0"/>
+				<mass value=".17"/>
+				<inertia ixx="0.001"  ixy="0"  ixz="0" iyy="0.001" iyz="0" izz="0.001"/>
+			</inertial>
+			<collision>
+				<origin xyz="${-chassis_length/2 + 2*lidar_radius} 0 ${chassis_height/2}"/>
+				<geometry>
+					<cylinder radius="${lidar_radius}" length=".06"/>
+				</geometry>
+			</collision>
+			<visual>
+				<origin xyz = "0 0 ${chassis_height/2}" rpy="0 0 0"/>
+				<geometry>
+					<cylinder radius="${lidar_radius}" length=".06"/>
+				</geometry>
+				<material name="Gray">
+					<color rgba="0.5 0.5 0.5 1.0"/>
+				</material>
+			</visual>
+		</link>
+		<!--create the joint that the lidar_link will be bound to with the base being the base_link-->
+		<joint name="lidar_joint" type="fixed">
+		<!--^^make joint continuous to mimic spinning lidar?-->
+			<parent link="chassis"/>
+			<child link="lidar_link"/>
+			<origin xyz="${-chassis_length/2 + lidar_radius} 0 ${chassis_height/2+.02}" rpy="0 0 0"/>
+		</joint>
+	</xacro:unless>
+	<xacro:if value="$(arg sim_mode)">
+		<!--adding gazebo plugins to the sim-->
+		<gazebo reference="lidar_link">
+			<sensor name="lidar" type="ray">
+				<always_on>true</always_on>
+				<visualize>true</visualize>
+				<update_rate>5</update_rate>
+				<ray>
+					<scan>
+						<horizontal>
+							<samples>8000</samples>
+							<resolution>1</resolution>
+							<!--min and max angles are in radians-->
+							<min_angle>0.0</min_angle>
+							<max_angle>6.28</max_angle>
+						</horizontal>
+					</scan>
+					<range>
+						<min>0.12</min>
+						<max>4</max>
 						<resolution>1</resolution>
-						<!--min and max angles are in radians-->
-						<min_angle>0.0</min_angle>
-						<max_angle>6.28</max_angle>
-					</horizontal>
-				</scan>
-				<range>
-					<min>0.12</min>
-					<max>4</max>
-					<resolution>1</resolution>
-				</range>
-				<noise>
-					<type>gaussian</type>
-					<mean>0.0</mean>
-					<stddev>0.01</stddev>
-				</noise>
-			</ray>
-			<plugin name="scan" filename="libgazebo_ros_ray_sensor.so">
-				<ros>
-					<namespace>/demo</namespace>
-					<remapping>~/out:=scan</remapping>
-				</ros>
-				<output_type>sensor_msgs/LaserScan</output_type>
-				<frame_name>lidar_link</frame_name>
-			</plugin>
-		</sensor>
-	</gazebo>
+					</range>
+					<noise>
+						<type>gaussian</type>
+						<mean>0.0</mean>
+						<stddev>0.01</stddev>
+					</noise>
+				</ray>
+				<plugin name="scan" filename="libgazebo_ros_ray_sensor.so">
+					<ros>
+						<namespace>/demo</namespace>
+						<remapping>~/out:=scan</remapping>
+					</ros>
+					<output_type>sensor_msgs/LaserScan</output_type>
+					<frame_name>lidar_link</frame_name>
+				</plugin>
+			</sensor>
+		</gazebo>
+	</xacro:if>
 </robot>

File: src/icarus_pi/description/robot_core.xacro (robot description, xacro)
@@ -68,7 +68,7 @@
 	    </link>
 	</xacro:macro>
-	<xacro:wheel prefix="frontLeft" x_reflect="-1" y_reflect="-1"/>
-	<xacro:wheel prefix="frontRight" x_reflect="-1" y_reflect="1"/>
-	<xacro:wheel prefix="backLeft" x_reflect="1" y_reflect="-1"/>
-	<xacro:wheel prefix="backRight" x_reflect="1" y_reflect="1"/>
+	<xacro:wheel prefix="backRight" x_reflect="-1" y_reflect="-1"/>
+	<xacro:wheel prefix="backLeft" x_reflect="-1" y_reflect="1"/>
+	<xacro:wheel prefix="frontRight" x_reflect="1" y_reflect="-1"/>
+	<xacro:wheel prefix="frontLeft" x_reflect="1" y_reflect="1"/>
 </robot>

Commit message: Fixed Lidar Not Rendering

File: src/icarus_pi/description/lidar.xacro (robot description, xacro)
@@ -1,74 +1,70 @@
 <?xml version="1.0"?>
 <robot xmlns:xacro="http://www.ros.org/wiki/xacro" >
-	<xacro:unless value="$(arg sim_mode)">
-		<!--lidar intrinsics-->
-		<link name="lidar_link">
-			<inertial>
-				<origin xyz="${-chassis_length/2 + 2*lidar_radius} 0 ${chassis_height/2}" rpy="0 0 0"/>
-				<mass value=".17"/>
-				<inertia ixx="0.001"  ixy="0"  ixz="0" iyy="0.001" iyz="0" izz="0.001"/>
-			</inertial>
-			<collision>
-				<origin xyz="${-chassis_length/2 + 2*lidar_radius} 0 ${chassis_height/2}"/>
-				<geometry>
-					<cylinder radius="${lidar_radius}" length=".06"/>
-				</geometry>
-			</collision>
-			<visual>
-				<origin xyz = "0 0 ${chassis_height/2}" rpy="0 0 0"/>
-				<geometry>
-					<cylinder radius="${lidar_radius}" length=".06"/>
-				</geometry>
-				<material name="Gray">
-					<color rgba="0.5 0.5 0.5 1.0"/>
-				</material>
-			</visual>
-		</link>
-		<!--create the joint that the lidar_link will be bound to with the base being the base_link-->
-		<joint name="lidar_joint" type="fixed">
-		<!--^^make joint continuous to mimic spinning lidar?-->
-			<parent link="chassis"/>
-			<child link="lidar_link"/>
-			<origin xyz="${-chassis_length/2 + lidar_radius} 0 ${chassis_height/2+.02}" rpy="0 0 0"/>
-		</joint>
-	</xacro:unless>
-	<xacro:if value="$(arg sim_mode)">
-		<!--adding gazebo plugins to the sim-->
-		<gazebo reference="lidar_link">
-			<sensor name="lidar" type="ray">
-				<always_on>true</always_on>
-				<visualize>true</visualize>
-				<update_rate>5</update_rate>
-				<ray>
-					<scan>
-						<horizontal>
-							<samples>8000</samples>
-							<resolution>1</resolution>
-							<!--min and max angles are in radians-->
-							<min_angle>0.0</min_angle>
-							<max_angle>6.28</max_angle>
-						</horizontal>
-					</scan>
-					<range>
-						<min>0.12</min>
-						<max>4</max>
+	<!--lidar intrinsics-->
+	<link name="lidar_link">
+		<inertial>
+			<origin xyz="${-chassis_length/2 + 2*lidar_radius} 0 ${chassis_height/2}" rpy="0 0 0"/>
+			<mass value=".17"/>
+			<inertia ixx="0.001"  ixy="0"  ixz="0" iyy="0.001" iyz="0" izz="0.001"/>
+		</inertial>
+		<collision>
+			<origin xyz="${-chassis_length/2 + 2*lidar_radius} 0 ${chassis_height/2}"/>
+			<geometry>
+				<cylinder radius="${lidar_radius}" length=".06"/>
+			</geometry>
+		</collision>
+		<visual>
+			<origin xyz = "0 0 ${chassis_height/2}" rpy="0 0 0"/>
+			<geometry>
+				<cylinder radius="${lidar_radius}" length=".06"/>
+			</geometry>
+			<material name="Gray">
+				<color rgba="0.5 0.5 0.5 1.0"/>
+			</material>
+		</visual>
+	</link>
+	<!--create the joint that the lidar_link will be bound to with the base being the base_link-->
+	<joint name="lidar_joint" type="fixed">
+	<!--^^make joint continuous to mimic spinning lidar?-->
+		<parent link="chassis"/>
+		<child link="lidar_link"/>
+		<origin xyz="${-chassis_length/2 + lidar_radius} 0 ${chassis_height/2+.02}" rpy="0 0 0"/>
+	</joint>
+	<!--adding gazebo plugins to the sim-->
+	<gazebo reference="lidar_link">
+		<sensor name="lidar" type="ray">
+			<always_on>true</always_on>
+			<visualize>true</visualize>
+			<update_rate>5</update_rate>
+			<ray>
+				<scan>
+					<horizontal>
+						<samples>8000</samples>
 						<resolution>1</resolution>
-					</range>
-					<noise>
-						<type>gaussian</type>
-						<mean>0.0</mean>
-						<stddev>0.01</stddev>
-					</noise>
-				</ray>
-				<plugin name="scan" filename="libgazebo_ros_ray_sensor.so">
-					<ros>
-						<namespace>/demo</namespace>
-						<remapping>~/out:=scan</remapping>
-					</ros>
-					<output_type>sensor_msgs/LaserScan</output_type>
-					<frame_name>lidar_link</frame_name>
-				</plugin>
-			</sensor>
-		</gazebo>
-	</xacro:if>
+						<!--min and max angles are in radians-->
+						<min_angle>0.0</min_angle>
+						<max_angle>6.28</max_angle>
+					</horizontal>
+				</scan>
+				<range>
+					<min>0.12</min>
+					<max>4</max>
+					<resolution>1</resolution>
+				</range>
+				<noise>
+					<type>gaussian</type>
+					<mean>0.0</mean>
+					<stddev>0.01</stddev>
+				</noise>
+			</ray>
+			<plugin name="scan" filename="libgazebo_ros_ray_sensor.so">
+				<ros>
+					<namespace>/demo</namespace>
+					<remapping>~/out:=scan</remapping>
+				</ros>
+				<output_type>sensor_msgs/LaserScan</output_type>
+				<frame_name>lidar_link</frame_name>
+			</plugin>
+		</sensor>
+	</gazebo>
 </robot>

Commit message: lidar location fix

File: src/icarus_pi/description/lidar.xacro (robot description, xacro)
@@ -4,10 +4,10 @@
 	<link name="lidar_link">
 		<inertial>
-			<origin xyz="${-chassis_length/2 + 2*lidar_radius} 0 ${chassis_height/2}" rpy="0 0 0"/>
+			<origin xyz = "0 0 0" rpy="0 0 0"/>
 			<mass value=".17"/>
 			<inertia ixx="0.001"  ixy="0"  ixz="0" iyy="0.001" iyz="0" izz="0.001"/>
 		</inertial>
 		<collision>
-			<origin xyz="${-chassis_length/2 + 2*lidar_radius} 0 ${chassis_height/2}"/>
+			<origin xyz = "0 0 0"/>
 			<geometry>
 				<cylinder radius="${lidar_radius}" length=".06"/>
@@ -15,5 +15,5 @@
 		</collision>
 		<visual>
-			<origin xyz = "0 0 ${chassis_height/2}" rpy="0 0 0"/>
+			<origin xyz = "0 0 0" rpy="0 0 0"/>
 			<geometry>
 				<cylinder radius="${lidar_radius}" length=".06"/>
@@ -29,5 +29,5 @@
 		<parent link="chassis"/>
 		<child link="lidar_link"/>
-		<origin xyz="${-chassis_length/2 + lidar_radius} 0 ${chassis_height/2+.02}" rpy="0 0 0"/>
+		<origin xyz="${lidar_radius} 0 ${chassis_height+.03}" rpy="0 0 0"/>
 	</joint>
 	<!--adding gazebo plugins to the sim-->

Commit message: corrected incorrect odom reading issue

File: src/icarus_pi/description/lidar.xacro (robot description, xacro)
@@ -27,5 +27,4 @@
 		<!--create the joint that the lidar_link will be bound to with the base being the base_link-->
 		<joint name="lidar_joint" type="fixed">
-		<!--^^make joint continuous to mimic spinning lidar?-->
 			<parent link="chassis"/>
 			<child link="lidar_link"/>

File: src/icarus_pi/description/robot_core.xacro (robot description, xacro)
@@ -42,9 +42,9 @@
     </gazebo>
     <!-- wheels -->
-	<xacro:macro name="wheel" params="prefix x_reflect y_reflect">
+	<xacro:macro name="wheel" params="prefix x_reflect y_reflect rotate">
         <joint name="${prefix}_joint" type="continuous">
             <parent link="base_link"/>
             <child link="${prefix}_link"/>
-            <origin xyz="${x_reflect*wheel_xoff} ${y_reflect*(chassis_width/2 + wheel_ygap)} ${-wheel_zoff}" rpy="-${pi/2} 0 0"/>
+            <origin xyz="${x_reflect*wheel_xoff} ${y_reflect*(chassis_width/2 + wheel_ygap)} ${-wheel_zoff}" rpy="-${pi/2} 0 ${rotate}"/>
             <axis xyz="0 0 1"/>
         </joint>
@@ -68,7 +68,7 @@
 	    </link>
 	</xacro:macro>
-	<xacro:wheel prefix="backRight" x_reflect="-1" y_reflect="-1"/>
-	<xacro:wheel prefix="backLeft" x_reflect="-1" y_reflect="1"/>
-	<xacro:wheel prefix="frontRight" x_reflect="1" y_reflect="-1"/>
-	<xacro:wheel prefix="frontLeft" x_reflect="1" y_reflect="1"/>
+	<xacro:wheel prefix="backRight" x_reflect="1" y_reflect="1" rotate="${pi}"/>
+	<xacro:wheel prefix="backLeft" x_reflect="1" y_reflect="-1" rotate="${pi}"/>
+	<xacro:wheel prefix="frontRight" x_reflect="-1" y_reflect="1" rotate="${pi}"/>
+	<xacro:wheel prefix="frontLeft" x_reflect="-1" y_reflect="-1" rotate="${pi}"/>
 </robot>

Commit message: fixed angular drift accumulated error

File: src/icarus_pi/description/lidar.xacro (robot description, xacro)
@@ -27,5 +27,5 @@
 	<joint name="lidar_joint" type="fixed">
 	<!--^^make joint continuous to mimic spinning lidar?-->
-		<parent link="chassis"/>
+		<parent link="base_link"/>
 		<child link="lidar_link"/>
 		<origin xyz="${lidar_radius} 0 ${chassis_height + 0.03}" rpy="0 0 0"/>
@@ -61,5 +61,4 @@
 			<plugin name="scan" filename="libgazebo_ros_ray_sensor.so">
 				<ros>
-					<namespace>/demo</namespace>
 					<remapping>~/out:=scan</remapping>
 				</ros>

File: src/icarus_pi/description/robot_core.xacro (robot description, xacro)
@@ -44,5 +44,5 @@
 	<xacro:macro name="wheel" params="prefix x_reflect y_reflect rotate">
         <xacro:if value="$(arg sim_mode)">
-            <joint name="${prefix}_joint" type="fixed">
+            <joint name="${prefix}_joint" type="continuous">
                 <parent link="base_link"/>
                 <child link="${prefix}_link"/>

File: src/icarus_pi/description/robot_dimensions.xacro (robot description, xacro)
@@ -3,5 +3,5 @@
     <!--constants to use for the robot dimensions-->
     <xacro:property name="chassis_length" value = ".18"/>
-    <xacro:property name="chassis_width" value = ".203"/>
+    <xacro:property name="chassis_width" value = ".19"/>
     <xacro:property name="chassis_height" value = ".16"/>
     <xacro:property name="chassis_mass" value = "1"/>

Commit message: odom parameter tuning

File: src/icarus_pi/description/lidar.xacro (robot description, xacro)
@@ -27,5 +27,5 @@
 	<joint name="lidar_joint" type="fixed">
 	<!--^^make joint continuous to mimic spinning lidar?-->
-		<parent link="base_link"/>
+		<parent link="chassis"/>
 		<child link="lidar_link"/>
 		<origin xyz="${lidar_radius} 0 ${chassis_height + 0.03}" rpy="0 0 0"/>

File: src/icarus_pi/description/robot_core.xacro (robot description, xacro)
@@ -43,5 +43,4 @@
     <!-- wheels -->
 	<xacro:macro name="wheel" params="prefix x_reflect y_reflect rotate">
-        <xacro:if value="$(arg sim_mode)">
             <joint name="${prefix}_joint" type="continuous">
                 <parent link="base_link"/>
@@ -50,13 +49,4 @@
                 <axis xyz="0 0 1"/>
             </joint>
-        </xacro:if>
-        <xacro:unless value="$(arg use_ros2_control)">
-            <joint name="${prefix}_joint" type="continuous">
-                <parent link="base_link"/>
-                <child link="${prefix}_link"/>
-                <origin xyz="${x_reflect*wheel_xoff} ${y_reflect*(chassis_width/2 + wheel_ygap)} ${-wheel_zoff}" rpy="-${pi/2} 0 ${rotate}"/>
-                <axis xyz="0 0 1"/>
-            </joint>
-        </xacro:unless>
         <link name ="${prefix}_link">
 			<collision>

File: src/icarus_pi/description/robot_dimensions.xacro (robot description, xacro)
@@ -2,6 +2,6 @@
 <robot xmlns:xacro="http://www.ros.org/wiki/xacro" >
     <!--constants to use for the robot dimensions-->
-    <xacro:property name="chassis_length" value = ".18"/>
-    <xacro:property name="chassis_width" value = ".19"/>
+    <xacro:property name="chassis_length" value = ".194"/>
+    <xacro:property name="chassis_width" value = ".17"/>
     <xacro:property name="chassis_height" value = ".16"/>
     <xacro:property name="chassis_mass" value = "1"/>

Commit message: flipped robot direction and wheels

File: src/icarus_pi/description/lidar.xacro (robot description, xacro)
@@ -29,5 +29,5 @@
 		<parent link="chassis"/>
 		<child link="lidar_link"/>
-		<origin xyz="${lidar_radius} 0 ${chassis_height + 0.03}" rpy="0 0 0"/>
+		<origin xyz="${chassis_length-lidar_radius} 0 ${chassis_height + 0.03}" rpy="0 0 0"/>
 	</joint>
 	<!--adding gazebo plugins to the sim-->

File: src/icarus_pi/description/robot_core.xacro (robot description, xacro)
@@ -44,6 +44,6 @@
             <parent link="base_link"/>
             <child link="${prefix}_link"/>
-            <origin xyz="${x_reflect*wheel_xoff} ${y_reflect*(chassis_width/2 + wheel_ygap)} ${-wheel_zoff}" rpy="-${pi/2} 0 ${rotate}"/>
-            <axis xyz="0 0 1"/>
+            <origin xyz="${x_reflect*wheel_xoff} ${y_reflect*(chassis_width/2 + wheel_ygap)} ${-wheel_zoff}" rpy="${y_reflect*-pi/2} 0 0"/>
+            <axis xyz="0 0 ${y_reflect}"/>
         </joint>
         <link name ="${prefix}_link">
@@ -66,8 +66,8 @@
 	    </link>
 	</xacro:macro>
-	<xacro:wheel prefix="backRight" x_reflect="1" y_reflect="1" rotate="${pi}"/>
-	<xacro:wheel prefix="backLeft" x_reflect="1" y_reflect="-1" rotate="${pi}"/>
-	<xacro:wheel prefix="frontRight" x_reflect="-1" y_reflect="1" rotate="${pi}"/>
-	<xacro:wheel prefix="frontLeft" x_reflect="-1" y_reflect="-1" rotate="${pi}"/>
+	<xacro:wheel prefix="backRight" x_reflect="-1" y_reflect="-1" rotate="${pi}"/>
+	<xacro:wheel prefix="backLeft" x_reflect="-1" y_reflect="1" rotate="${pi}"/>
+	<xacro:wheel prefix="frontRight" x_reflect="1" y_reflect="-1" rotate="${pi}"/>
+	<xacro:wheel prefix="frontLeft" x_reflect="1" y_reflect="1" rotate="${pi}"/>
     <gazebo reference="backRight_link">
         <material>Gazebo/ZincYellow</material>

Commit message: flipped the lidar to match with its pre-defined hardware axis

File: src/icarus_pi/description/lidar.xacro (robot description, xacro)
@@ -29,5 +29,5 @@
 		<parent link="chassis"/>
 		<child link="lidar_link"/>
-		<origin xyz="${chassis_length-lidar_radius} 0 ${chassis_height + 0.03}" rpy="0 0 0"/>
+		<origin xyz="${chassis_length-lidar_radius} 0 ${chassis_height + 0.03}" rpy="0 0 ${pi}"/>
 	</joint>
 	<!--adding gazebo plugins to the sim-->
