Commit message: Updated Robot Core Wheel Positions

File: src/icarus_pi/description/gazebo_robot_core.xacro (robot description, xacro)
@@ -44,5 +44,5 @@
             <parent link="base_link"/>
             <child link="${prefix}_link"/>
-            <origin xyz="${x_reflect*wheel_xoff} ${y_reflect*(chassis_width/2 + wheel_ygap)} ${-wheel_zoff}" rpy="-${pi/2} 0 0"/>
+               <origin xyz="${x_reflect*wheel_xoff} ${y_reflect*(chassis_width/2 + wheel_ygap)} ${-wheel_zoff}" rpy="-${pi/2} 0 ${rotate}"/>
             <axis xyz="0 0 1"/>
         </joint>
